File: Hardware/Hardware_électronique/Auxiliairy_board/PCB_Moteur/Inverter_KiCAD/pwrSupply.kicad_sch (KiCad schematic)
At the start: 11 parts, among them J4 Conn_01x02_Pin, U503 AZ1117-3.3

Commit message: Add files via upload
Parts:
- added C22: 10u, symbol Device:C
- added C23: 47u, symbol Device:C
- added C24: 0.022u, symbol Device:C
- added C25: 4700p, symbol Device:C
- added Converter_DCDC_WPMDH1302401: ~, Custom:Converter_DCDC, symbol Custom:Converter_DCDC
- added R16: 287k, symbol Device:R
- added R17: 34k, symbol Device:R
- added R18: 1.91k, symbol Device:R
Connections:
- net ISO_GND is gone; now on net ISO_GRND: C501.2, C502.2, R501.2, R502.2, R503.2, U503.1 (GND)
- net ISO_15V: now also C23.1, C24.1, Converter_DCDC_WPMDH1302401.7 (Vout), R17.1
- net at J4.1 (Pin_1): now also C22.1, Converter_DCDC_WPMDH1302401.1 (Vin), R16.1
- net ISO_GRND: now reaches F501.2
- net ISO_GRND: now also C22.2, C23.2, C25.2, Converter_DCDC_WPMDH1302401.4 (AGND), Converter_DCDC_WPMDH1302401.8 (PGND), R18.2
- new net: Converter_DCDC_WPMDH1302401.2 (RON), Converter_DCDC_WPMDH1302401.3 (EN), R16.2
- new net: C25.1, Converter_DCDC_WPMDH1302401.5 (SS)
- new net: C24.2, Converter_DCDC_WPMDH1302401.6 (FB), R17.2, R18.1
Other:
- moved on the sheet: D501, D502, D503, F501, R501, R502, R503

Commit message: Add files via upload
Parts:
- added J5: 173010542, Buck_5V_173010542:173010542, symbol 173010542_5V_Buck:173010542
Connections:
- net ISO_15V: now also J5.1 (VIN)
- net ISO_5V: now also J5.3 (VOUT)
- net ISO_GRND: now also J5.2 (GND)
Other:
- note added: "LDO Regalator Based on Wurth 173010542 5V for LIDAR Vin : 7V-42V Vout : 5V Max : 1A"
- note removed: "Max output current : 1A"
Changed lines of the file:
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@@
-	(wire
-		(pts
-			(xy 123.19 36.83) (xy 125.73 36.83)
-		)
-		(stroke
-			(width 0)
-			(type default)
-		)
-	)
 	(wire
 		(pts
@@
 	(wire
 		(pts
+			(xy 135.89 48.26) (xy 135.89 50.8)
+		)
+		(stroke
+			(width 0)
+			(type default)
+		)
+	)
+	(wire
+		(pts
 			(xy 77.47 39.37) (xy 77.47 40.64)
 		)
@@
 	(wire
 		(pts
+			(xy 144.78 40.64) (xy 149.86 40.64)
+		)
+		(stroke
+			(width 0)
+			(type default)
+		)
+	)
+	(wire
+		(pts
 			(xy 49.53 41.91) (xy 46.99 41.91)
 		)
@@
 	(wire
 		(pts
+			(xy 123.19 40.64) (xy 127 40.64)
+		)
+		(stroke
+			(width 0)
+			(type default)
+		)
+	)
+	(wire
+		(pts
 			(xy 27.94 39.37) (xy 38.1 39.37)
 		)
@@
 	(wire
 		(pts
-			(xy 151.13 36.83) (xy 148.59 36.83)
-		)
-		(stroke
-			(width 0)
-			(type default)
-		)
-	)
-	(wire
-		(pts
 			(xy 66.04 107.95) (xy 67.31 107.95)
 		)
@@
 		(pts
 			(xy 92.71 39.37) (xy 92.71 45.72)
-		)
-		(stroke
-			(width 0)
-			(type default)
-		)
-	)
-	(wire
-		(pts
-			(xy 137.16 46.99) (xy 137.16 44.45)
 		)
 		(stroke
@@
 	)
 	(rectangle
-		(start 105.41 13.97)
-		(end 179.07 66.04)
+		(start 107.95 17.78)
+		(end 172.72 63.5)
 		(stroke
 			(width 0)
@@
 		(fill
 			(type none)
+		)
+	)
+	(text "LDO Regalator\nBased on Wurth 173010542\n5V for LIDAR\nVin : 7V-42V\nVout : 5V\nMax : 1A"
+		(exclude_from_sim no)
+		(at 117.856 30.988 0)
+		(effects
+			(font
+				(size 1.27 1.27)
+			)
+			(justify left bottom)
 		)
 	)
@@
 		(exclude_from_sim no)
 		(at 184.15 21.59 0)
-		(effects
-			(font
-				(size 1.27 1.27)
-			)
-			(justify left bottom)
-		)
-	)
-	(text "Max output current : 1A"
-		(exclude_from_sim no)
-		(at 106.172 17.78 0)
 		(effects
 			(font
@@
 		)
 	)
-	(hierarchical_label "ISO_5V"
-		(shape input)
-		(at 151.13 36.83 0)
-		(fields_autoplaced yes)
-		(effects
-			(font
-				(size 1.27 1.27)
-			)
-			(justify left)
-		)
-	)
 	(hierarchical_label "ISO_GND"
 		(shape input)
@@
 	(hierarchical_label "ISO_15V"
 		(shape input)
-		(at 123.19 36.83 180)
-		(fields_autoplaced yes)
-		(effects
-			(font
-				(size 1.27 1.27)
-			)
-			(justify right)
-		)
-	)
-	(hierarchical_label "ISO_15V"
-		(shape input)
 		(at 93.98 39.37 0)
 		(fields_autoplaced yes)
@@
 		)
 	)
-	(hierarchical_label "ISO_GND"
-		(shape input)
-		(at 137.16 46.99 270)
-		(fields_autoplaced yes)
-		(effects
-			(font
-				(size 1.27 1.27)
-			)
-			(justify right)
-		)
-	)
 	(hierarchical_label "ISO_5V"
 		(shape input)
@@
 		(shape input)
 		(at 50.8 99.06 180)
+		(fields_autoplaced yes)
+		(effects
+			(font
+				(size 1.27 1.27)
+			)
+			(justify right)
+		)
+	)
+	(hierarchical_label "ISO_5V"
+		(shape input)
+		(at 149.86 40.64 0)
+		(fields_autoplaced yes)
+		(effects
+			(font
+				(size 1.27 1.27)
+			)
+			(justify left)
+		)
+	)
+	(hierarchical_label "ISO_GND"
+		(shape input)
+		(at 135.89 50.8 270)
+		(fields_autoplaced yes)
+		(effects
+			(font
+				(size 1.27 1.27)
+			)
+			(justify right)
+		)
+	)
+	(hierarchical_label "ISO_15V"
+		(shape input)
+		(at 123.19 40.64 180)
 		(fields_autoplaced yes)
 		(effects
@@
 					(unit 1)
 				)
+			)
+		)
+	)
+	(symbol
+		(lib_id "173010542_5V_Buck:173010542")
+		(at 135.89 41.91 0)
+		(unit 1)
+		(exclude_from_sim no)
+		(in_bom yes)
+		(on_board yes)
+		(dnp no)
+		(fields_autoplaced yes)
+		(property "Reference" "J5"
+			(at 135.89 33.02 0)
+			(effects
+				(font
+					(size 1.524 1.524)
+				)
+			)
+		)
+		(property "Value" "173010542"
+			(at 135.89 35.56 0)
+			(effects
+				(font
+					(size 1.524 1.524)
+				)
+			)
+		)
+		(property "Footprint" "Buck_5V_173010542:173010542"
+			(at 134.62 29.21 0)
+			(effects
+				(font
+					(size 1.27 1.27)
+					(italic yes)
+				)
+				(hide yes)
+			)
+		)
+		(property "Datasheet" "https://www.we-online.com/components/products/datasheet/173010542.pdf"
+			(at 135.89 31.75 0)
+			(effects
+				(font
+					(size 1.27 1.27)
+					(italic yes)
+				)
+				(hide yes)
+			)
+		)
+		(property "Description" ""
+			(at 135.89 41.91 0)
+			(effects
+				(font
+					(size 1.27 1.27)
+				)
+				(hide yes)
+			)
+		)
+		(property "MPN" "173010542"
+			(at 135.89 41.91 0)
+			(effects
+				(font
+					(size 1.27 1.27)
+				)
+				(hide yes)
+			)
+		)
+		(pin "1"
+		)
+		(pin "2"
+		)
+		(pin "3"
+		)
+		(instances
+			(project "Inverter_KiCAD"
+				(path "/5e6c1e3f-0815-454a-8acb-8e3e2d064875/c44552c8-6743-4bce-b187-ccb6744e5f40"
+					(reference "J5")
+					(unit 1)
+				)
