File: Hardware/Hardware_électronique/Auxiliairy_board/PCB_Moteur/Inverter_KiCAD/pwrSupply.kicad_sch (KiCad schematic)
At the start: 20 parts, among them J4 Conn_01x02_Pin, J5 173010542, U503 AZ1117-3.3

Commit message: update schematic
Parts:
- removed C22: 10u, symbol Device:C
- removed C23: 47u, symbol Device:C
- removed C24: 22nF, symbol Device:C
- removed C25: 4.7nF, symbol Device:C
- removed C501: 10u, Capacitor_SMD:CP_Elec_4x5.4, symbol Device:C_Polarized
- removed C502: 22u, Capacitor_SMD:CP_Elec_5x5.4, symbol Device:C_Polarized
- removed Converter_DCDC_WPMDH1302401: ~, Custom:Converter_DCDC, symbol Custom:Converter_DCDC
- removed D501, D502, D503: Red LED, LED_SMD:LED_0603_1608Metric, symbol Device:LED
- removed F501: Fuse, Custom:0031.8201, symbol Device:Fuse
- removed J4: Conn_01x02_Pin, Connector_AMASS:AMASS_XT60PW-F_1x02_P7.20mm_Horizontal, symbol Connector:Conn_01x02_Pin
- removed J5: 173010542, Buck_5V_173010542:173010542, symbol 173010542_5V_Buck:173010542
- removed R16: 287k, symbol Device:R
- removed R17: 34k, symbol Device:R
- removed R18: 1.91k, symbol Device:R
- removed R501: 2k7, Resistor_SMD:R_0402_1005Metric, symbol Device:R_Small
- removed R502: 680, Resistor_SMD:R_0402_1005Metric, symbol Device:R_Small
- removed R503: 390, Resistor_SMD:R_0402_1005Metric, symbol Device:R_Small
- removed U503: AZ1117-3.3, Package_TO_SOT_SMD:SOT-223-3_TabPin2, symbol Regulator_Linear:AZ1117-3.3
Other:
- note removed: "LDO Regalator Based on Wurth 173010542 5V for LIDAR Vin : 7V-42V Vout : 5V Max : 1A"
- note removed: "LED power"
- note removed: "Max output current : 800mA -> uC -> hall sensors"
