File: Hardware/Hardware_électronique/Auxiliairy_board/PCB_Moteur/Inverter_KiCAD/Arm_IRF540NBbF.kicad_sch (KiCad schematic)
At the start: 33 parts, among them Q3 IRF540N, Q302 IRF540N, Q303 IRF540N, Q4 IRF540N, U10 MPRB2415S-6W, U2 MIC4606, U5 GO 10-SME/SP3, U9 MPRB2415S-6W

Commit message: Add files via upload
Parts:
- renumbered C2 to C1, C17 to C16, C20 to C19, C306 to C206, C309 to C209, C310 to C210, C311 to C211, C8 to C4, C9 to C5, C10 to C6, C11 to C7, D2 to D1, D302 to D202, D303 to D203, D6 to D4, D7 to D5, Q3 to Q1, Q4 to Q2, Q302 to Q202, Q303 to Q203, R2 to R1, R12 to R10, R13 to R11, R301 to R201, R302 to R202, R304 to R204, R305 to R205, R5 to R4, R8 to R7, U2 to U1, U5 to U4, U9 to U7, U10 to U8
Connections:
- net ARM_OUT: no longer U4.1 (IP+), U4.2 (IP+)
- net ARM_OUT_A: now also U4.1 (IP+), U4.2 (IP+)

Commit message: update schematic
Parts:
- removed C4, C5: 100u, Capacitor_SMD:CP_Elec_6.3x7.7, symbol Device:C_Polarized
- removed C6, C7: 22u, Capacitor_SMD:CP_Elec_5x5.4, symbol Device:C_Polarized
- removed D1: Green LED, LED_SMD:LED_0603_1608Metric, symbol Device:LED
- removed R1: 390, Resistor_SMD:R_0402_1005Metric, symbol Device:R_Small
- removed R201, R202, R4, R7: 170, Resistor_SMD:R_0402_1005Metric, symbol Device:R_Small
- removed U7, U8: MPRB2415S-6W, Custom:MPRB2415S, symbol Custom:MPRB2415S-6W
- added J1: Conn_02x02_Top_Bottom, Connector_Molex:Molex_Micro-Fit_3.0_43045-0400_2x02_P3.00mm_Horizontal, symbol Connector_Generic:Conn_02x02_Top_Bottom
Connections:
- net V_Out is gone; now on net ARM_OUT_A: U4.3 (IP-), U4.4 (IP-)
- net ARM_OUT_A: now also J1.1 (Pin_1); no longer C16.1, Q1.3 (S), Q2.2 (D), U1.10 (AHS), U4.1 (IP+), U4.2 (IP+)
- net GND: now also C209.2, C210.2, C211.2, R10.2, R11.2, R204.2, R205.2, U4.5 (GND), J1.2 (Pin_2)
- net ISO_GND: no longer C209.2, C210.2, C211.2, R10.2, R11.2, R204.2, R205.2, U4.5 (GND)
- net In_A_H: now also U1.6 (AHI)
- net In_A_L: now also U1.5 (ALI)
- net In_B_H: now also U1.3 (BHI)
- net In_B_L: now also U1.4 (BLI)
- net ARM_OUT_B renamed ARM_B
- net ARM_B: now also J1.3 (Pin_3)
- new net ARM_IN_A: C16.1, Q1.3 (S), Q2.2 (D), U1.10 (AHS), U4.1 (IP+), U4.2 (IP+)
- no-connect marks 0 -> 1
Other:
- note added: "ADD UREF"
- note removed: "Isolated Power Supply Input : 15V Output : 2x15V"
- note removed: "Vgs (5V -> 10V)"
- moved on the sheet: C1, C206, C209, C210, C211, Q1, Q2, Q202, Q203, U4
