File: Hardware/Hardware_électronique/Auxiliairy_board/PCB_Moteur/Inverter_KiCAD/pwrSupplyFiltering.kicad_sch (KiCad schematic)
At the start: 5 parts

Commit message: Add files via upload
Parts:
- added D2, D3, D6: Red LED, LED_SMD:LED_0603_1608Metric, symbol Device:LED
- added R2: 27k, Resistor_SMD:R_0402_1005Metric, symbol Device:R_Small
- added R3, R5, R6: 10k, Resistor_SMD:R_0402_1005Metric, symbol Device:R_Small
- added U2: 17791063215, Custom:17791063215, symbol Custom:17791063215
Connections:
- net GND: now also R2.2, R3.2, R5.2, R6.2, U2.7 (Vout_Gnd)
- new net: D6.1 (K), R6.1
- new net: D3.1 (K), R5.1
- new net: R2.1, U2.8 (FB)
- new net: D2.1 (K), R3.1
- new net 5V: U2.6 (Vout)
- new net ISO_15V: U2.2 (Vin)
- new net ISO_GND: U2.1 (Vin_GND)
- new net PwrEn: U2.3 (Ctrl)
- new net VSupply_AB: D3.2 (A)
- new net VSupply_BB: D2.2 (A)
- new net Vbus: D6.2 (A)
Other:
- note added: "Isolated power Supply 5V / 200mA"
- note added: "V_Power_LED"
- note added: "Vout = (82.5k + Rfb)/Rfb*1.24V"
