File: Hardware/Hardware_électronique/Auxiliairy_board/PCB_Moteur/Inverter_KiCAD/pwrSupply_5V.kicad_sch (KiCad schematic)
At the start: 2 parts, among them U701 17791063215

Commit message: Add files via upload
Parts:
- removed R701: 27k, Resistor_SMD:R_0402_1005Metric, symbol Device:R_Small
- removed U701: 17791063215, Custom:17791063215, symbol Custom:17791063215
Other:
- note removed: "Isolated power Supply 5V / 200mA"
- note removed: "Vout = (82.5k + Rfb)/Rfb*1.24V"
