File: Hardware/Hardware_électronique/Auxiliairy_board/PCB_Moteur/Inverter_KiCAD/Inverter_KiCAD.kicad_sch (KiCad schematic)
At the start: 69 parts, among them J1 Conn_02x02_Top_Bottom, J2 173010542, J3 Conn_02x05_Odd_Even, J4 Conn_01x02, J5 Conn_01x02, Q5 SQ2310ES, U1 MIC4606, U2 GO 10-SME/SP3, U3 GO 10-SME/SP3, U4 AZ1117-3.3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

Commit message: PCB motor oof
Parts:
- removed H110, H112: MountingHole_Pad, MountingHole:MountingHole_3.2mm_M3_Pad_Via, symbol Mechanical:MountingHole_Pad
Changed lines of the file:
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@@
 	)
 	(junction
-		(at 374.65 228.6)
-		(diameter 0)
-		(color 0 0 0 0)
-	)
-	(junction
 		(at 142.24 247.65)
 		(diameter 0)
@@
 	)
 	(junction
-		(at 400.05 228.6)
-		(diameter 0)
-		(color 0 0 0 0)
-	)
-	(junction
 		(at 252.73 195.58)
 		(diameter 0)
@@
 	(wire
 		(pts
-			(xy 400.05 223.52) (xy 389.89 223.52)
-		)
-		(stroke
-			(width 0)
-			(type default)
-		)
-	)
-	(wire
-		(pts
 			(xy 22.86 50.8) (xy 29.21 50.8)
 		)
@@
 	(wire
 		(pts
-			(xy 370.84 228.6) (xy 374.65 228.6)
-		)
-		(stroke
-			(width 0)
-			(type default)
-		)
-	)
-	(wire
-		(pts
 			(xy 77.47 45.72) (xy 80.01 45.72)
 		)
@@
 	(wire
 		(pts
-			(xy 374.65 233.68) (xy 374.65 228.6)
+			(xy 374.65 223.52) (xy 374.65 233.68)
 		)
 		(stroke
@@
 	(wire
 		(pts
-			(xy 400.05 228.6) (xy 400.05 223.52)
-		)
-		(stroke
-			(width 0)
-			(type default)
-		)
-	)
-	(wire
-		(pts
 			(xy 85.09 271.78) (xy 90.17 271.78)
 		)
@@
 	(wire
 		(pts
-			(xy 374.65 228.6) (xy 374.65 223.52)
-		)
-		(stroke
-			(width 0)
-			(type default)
-		)
-	)
-	(wire
-		(pts
 			(xy 113.03 130.81) (xy 113.03 133.35)
 		)
@@
 	)
 	(symbol
-		(lib_id "Mechanical:MountingHole_Pad")
-		(at 368.3 228.6 90)
-		(unit 1)
-		(exclude_from_sim no)
-		(in_bom yes)
-		(on_board yes)
-		(dnp no)
-		(property "Reference" "H110"
-			(at 364.49 226.06 90)
-			(effects
-				(font
-					(size 1.27 1.27)
-				)
-			)
-		)
-		(property "Value" "MountingHole_Pad"
-			(at 367.03 226.06 90)
-			(effects
-				(font
-					(size 1.27 1.27)
-				)
-				(hide yes)
-			)
-		)
-		(property "Footprint" "MountingHole:MountingHole_3.2mm_M3_Pad_Via"
-			(at 368.3 228.6 0)
-			(effects
-				(font
-					(size 1.27 1.27)
-				)
-				(hide yes)
-			)
-		)
-		(property "Datasheet" "~"
-			(at 368.3 228.6 0)
-			(effects
-				(font
-					(size 1.27 1.27)
-				)
-				(hide yes)
-			)
-		)
-		(property "Description" ""
-			(at 368.3 228.6 0)
-			(effects
-				(font
-					(size 1.27 1.27)
-				)
-				(hide yes)
-			)
-		)
-		(property "MFR" "-"
-			(at 368.3 228.6 0)
-			(effects
-				(font
-					(size 1.27 1.27)
-				)
-				(hide yes)
-			)
-		)
-		(pin "1"
-		)
-		(instances
-			(project "Inverter_KiCAD"
-				(path "/5e6c1e3f-0815-454a-8acb-8e3e2d064875"
-					(reference "H110")
-					(unit 1)
-				)
-			)
-		)
-	)
-	(symbol
 		(lib_id "Device:R_Small")
 		(at 320.04 228.6 0)
@@
 					(unit 1)
 				)
-			)
-		)
-	)
-	(symbol
-		(lib_id "Mechanical:MountingHole_Pad")
-		(at 387.35 223.52 90)
-		(unit 1)
-		(exclude_from_sim no)
-		(in_bom yes)
-		(on_board yes)
-		(dnp no)
-		(property "Reference" "H112"
-			(at 383.54 220.98 90)
-			(effects
-				(font
-					(size 1.27 1.27)
-				)
-			)
-		)
-		(property "Value" "MountingHole_Pad"
-			(at 386.08 220.98 90)
-			(effects
-				(font
-					(size 1.27 1.27)
-				)
-				(hide yes)
-			)
-		)
-		(property "Footprint" "MountingHole:MountingHole_3.2mm_M3_Pad_Via"
-			(at 387.35 223.52 0)
-			(effects
-				(font
-					(size 1.27 1.27)
-				)
-				(hide yes)
-			)
-		)
-		(property "Datasheet" "~"
-			(at 387.35 223.52 0)
-			(effects
-				(font
-					(size 1.27 1.27)
-				)
-				(hide yes)
-			)
-		)
-		(property "Description" ""
-			(at 387.35 223.52 0)
-			(effects
-				(font
-					(size 1.27 1.27)
-				)
-				(hide yes)
-			)
-		)
-		(property "MFR" "-"
-			(at 387.35 223.52 0)
-			(effects
-				(font
-					(size 1.27 1.27)
-				)
-				(hide yes)
-			)
-		)
-		(pin "1"
-		)
-		(instances
-			(project "Inverter_KiCAD"
-				(path "/5e6c1e3f-0815-454a-8acb-8e3e2d064875"
-					(reference "H112")
-					(unit 1)
-				)

Commit message: ey
Parts:
- BT1: footprint Connector_AMASS:AMASS_XT60-F_1x02_P7.20mm_Vertical -> Connector_AMASS:AMASS_XT60-M_1x02_P7.20mm_Vertical
Changed lines of the file:
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@@
 	)
 	(junction
-		(at 102.87 114.3)
-		(diameter 0)
-		(color 0 0 0 0)
-	)
-	(junction
 		(at 92.71 172.72)
 		(diameter 0)
@@
 	)
 	(junction
-		(at 49.53 129.54)
-		(diameter 0)
-		(color 0 0 0 0)
-	)
-	(junction
 		(at 58.42 172.72)
 		(diameter 0)
@@
 	)
 	(junction
-		(at 39.37 113.03)
-		(diameter 0)
-		(color 0 0 0 0)
-	)
-	(junction
 		(at 332.74 241.3)
 		(diameter 0)
@@
 	(wire
 		(pts
-			(xy 40.64 113.03) (xy 40.64 114.3)
-		)
-		(stroke
-			(width 0)
-			(type default)
-		)
-	)
-	(wire
-		(pts
-			(xy 48.26 129.54) (xy 49.53 129.54)
+			(xy 46.99 129.54) (xy 59.69 129.54)
 		)
 		(stroke
@@
 	(wire
 		(pts
-			(xy 38.1 114.3) (xy 38.1 113.03)
-		)
-		(stroke
-			(width 0)
-			(type default)
-		)
-	)
-	(wire
-		(pts
 			(xy 252.73 181.61) (xy 254 181.61)
 		)
@@
 	(wire
 		(pts
-			(xy 49.53 129.54) (xy 60.96 129.54)
-		)
-		(stroke
-			(width 0)
-			(type default)
-		)
-	)
-	(wire
-		(pts
 			(xy 320.04 222.25) (xy 320.04 226.06)
 		)
@@
 	(wire
 		(pts
-			(xy 104.14 114.3) (xy 104.14 115.57)
-		)
-		(stroke
-			(width 0)
-			(type default)
-		)
-	)
-	(wire
-		(pts
 			(xy 50.8 87.63) (xy 64.77 87.63)
 		)
@@
 	(wire
 		(pts
-			(xy 49.53 132.08) (xy 49.53 129.54)
-		)
-		(stroke
-			(width 0)
-			(type default)
-		)
-	)
-	(wire
-		(pts
-			(xy 49.53 127) (xy 49.53 129.54)
-		)
-		(stroke
-			(width 0)
-			(type default)
-		)
-	)
-	(wire
-		(pts
 			(xy 58.42 182.88) (xy 69.85 182.88)
 		)
@@
 	(wire
 		(pts
-			(xy 102.87 113.03) (xy 102.87 114.3)
-		)
-		(stroke
-			(width 0)
-			(type default)
-		)
-	)
-	(wire
-		(pts
 			(xy 46.99 260.35) (xy 46.99 261.62)
 		)
@@
 	(wire
 		(pts
-			(xy 39.37 113.03) (xy 40.64 113.03)
-		)
-		(stroke
-			(width 0)
-			(type default)
-		)
-	)
-	(wire
-		(pts
 			(xy 81.28 182.88) (xy 92.71 182.88)
 		)
@@
 	(wire
 		(pts
-			(xy 101.6 114.3) (xy 102.87 114.3)
-		)
-		(stroke
-			(width 0)
-			(type default)
-		)
-	)
-	(wire
-		(pts
 			(xy 215.9 187.96) (xy 237.49 187.96)
 		)
@@
 	(wire
 		(pts
-			(xy 102.87 114.3) (xy 104.14 114.3)
-		)
-		(stroke
-			(width 0)
-			(type default)
-		)
-	)
-	(wire
-		(pts
 			(xy 53.34 110.49) (xy 53.34 111.76)
 		)
@@
 	(wire
 		(pts
-			(xy 101.6 115.57) (xy 101.6 114.3)
-		)
-		(stroke
-			(width 0)
-			(type default)
-		)
-	)
-	(wire
-		(pts
 			(xy 165.1 257.81) (xy 168.91 257.81)
 		)
@@
 	(wire
 		(pts
-			(xy 48.26 132.08) (xy 49.53 132.08)
-		)
-		(stroke
-			(width 0)
-			(type default)
-		)
-	)
-	(wire
-		(pts
 			(xy 168.91 269.24) (xy 182.88 269.24)
 		)
@@
 	(wire
 		(pts
-			(xy 38.1 113.03) (xy 39.37 113.03)
-		)
-		(stroke
-			(width 0)
-			(type default)
-		)
-	)
-	(wire
-		(pts
 			(xy 106.68 64.77) (xy 119.38 64.77)
 		)
@@
 	(wire
 		(pts
-			(xy 48.26 127) (xy 49.53 127)
-		)
-		(stroke
-			(width 0)
-			(type default)
-		)
-	)
-	(wire
-		(pts
 			(xy 92.71 181.61) (xy 92.71 182.88)
 		)
@@
 	)
 	(rectangle
-		(start 15.24 13.97)
-		(end 193.04 210.82)
-		(stroke
-			(width 1)
-			(type default)
-		)
-		(fill
-			(type color)
-			(color 255 246 235 1)
-		)
-	)
-	(rectangle
 		(start 303.53 168.91)
 		(end 400.05 205.74)
@@
 	)
 	(label "ARM_IN_A"
-		(at 60.96 129.54 180)
+		(at 59.69 129.54 180)
 		(fields_autoplaced yes)
 		(effects
@@
 	)
 	(symbol
+		(lib_name "CSD86350Q5D_1")
 		(lib_id "CSD87351Q5D:CSD86350Q5D")
 		(at 38.1 129.54 0)
@@
 		)
 		(property "Footprint" "CSD87351Q5D:DQY0008A"
-			(at 38.1 129.54 0)
+			(at 52.832 116.586 0)
 			(effects
 				(font
@@
 		)
 		(property "Datasheet" "CSD86350Q5D"
-			(at 38.1 129.54 0)
+			(at 47.752 118.618 0)
 			(effects
 				(font
@@
 		)
 		(property "Footprint" "CSD87351Q5D:DQY0008A"
-			(at 101.6 130.81 0)
+			(at 110.998 118.872 0)
 			(effects
 				(font
@@
 		)
 		(property "Datasheet" "CSD86350Q5D"
-			(at 101.6 130.81 0)
+			(at 110.998 120.904 0)
 			(effects
 				(font
@@
 			)
 		)
-		(property "Footprint" "Connector_AMASS:AMASS_XT60-F_1x02_P7.20mm_Vertical"
+		(property "Footprint" "Connector_AMASS:AMASS_XT60-M_1x02_P7.20mm_Vertical"
 			(at 22.86 242.316 90)
 			(effects
@@
 	(symbol
 		(lib_id "power:VBUS")
-		(at 39.37 113.03 0)
+		(at 38.1 114.3 0)
 		(unit 1)
 		(exclude_from_sim no)
@@
 		(fields_autoplaced yes)
 		(property "Reference" "#PWR048"
-			(at 39.37 116.84 0)
+			(at 38.1 118.11 0)
 			(effects
 				(font
@@
 		)
 		(property "Value" "VBUS"
-			(at 39.37 107.95 0)
+			(at 38.1 109.22 0)
 			(effects
 				(font
@@
 		)
 		(property "Footprint" ""
-			(at 39.37 113.03 0)
+			(at 38.1 114.3 0)
 			(effects
 				(font
@@
 		)
 		(property "Datasheet" ""
-			(at 39.37 113.03 0)
+			(at 38.1 114.3 0)
 			(effects
 				(font
@@
 		)
 		(property "Description" "Power symbol creates a global label with name \"VBUS\""
-			(at 39.37 113.03 0)
+			(at 38.1 114.3 0)
 			(effects
 				(font
@@
 	(symbol
 		(lib_id "power:VBUS")
-		(at 102.87 113.03 0)
+		(at 101.6 115.57 0)
 		(unit 1)
 		(exclude_from_sim no)
@@
 		(fields_autoplaced yes)
 		(property "Reference" "#PWR047"
-			(at 102.87 116.84 0)
+			(at 101.6 119.38 0)
 			(effects
 				(font
@@
 		)
 		(property "Value" "VBUS"
-			(at 102.87 107.95 0)
+			(at 101.6 110.49 0)
 			(effects
 				(font
@@
 		)
 		(property "Footprint" ""
-			(at 102.87 113.03 0)
+			(at 101.6 115.57 0)
 			(effects
 				(font
@@
 		)
 		(property "Datasheet" ""
-			(at 102.87 113.03 0)
+			(at 101.6 115.57 0)
 			(effects
 				(font
@@
 		)
 		(property "Description" "Power symbol creates a global label with name \"VBUS\""
-			(at 102.87 113.03 0)
+			(at 101.6 115.57 0)
 			(effects
 				(font

Commit message: hello
Parts:
- removed C11, C12: 220u, Capacitor_SMD:CP_Elec_10x10.5, symbol Device:C_Polarized

Commit message: commitment
Parts:
- R26: value 287k -> 100k
- R27: value 1.91k -> 4.3k
- R28: value 34k -> 36k
Other:
- note added: "SOULEVER PATE 3 AVANT DE SOUDER"
- moved on the sheet: J4, J5, Q5, R11, R12
