File: Hardware/Hardware_électronique/Auxiliairy_board/PCB_Moteur/Inverter_KiCAD/Inverter_KiCAD.kicad_pcb (KiCad board)
At the start: 4 copper layers, 1 part

Commit message: deut routage
Parts:
- added C10: 1.5m, Capacitor_THT:CP_Radial_D35.0mm_P10.00mm_SnapIn, F.Cu at (116.0, 135.3)
- added C11: 1.5m, Capacitor_THT:CP_Radial_D35.0mm_P10.00mm_SnapIn, F.Cu at (153.0, 58.0)
- added C12: 1.5m, Capacitor_THT:CP_Radial_D35.0mm_P10.00mm_SnapIn, F.Cu at (153.0, 136.0)
- added C1201: 100n, Capacitor_SMD:C_0402_1005Metric, F.Cu at (181.0, 100.0)
- added C13: 4.7n, Capacitor_SMD:C_0402_1005Metric, F.Cu at (190.2, 65.7)
- added C14: 4.7n, Capacitor_SMD:C_0402_1005Metric, F.Cu at (189.8, 69.5)
- added C15: 4.7n, Capacitor_SMD:C_0402_1005Metric, F.Cu at (189.8, 70.8)
- added C16: 10n, Capacitor_SMD:C_0402_1005Metric, F.Cu at (177.2, 67.5)
- added C17: 10u, Capacitor_SMD:CP_Elec_4x5.4, F.Cu at (184.2, 111.5)
- added C18: 22u, Capacitor_SMD:CP_Elec_5x5.4, F.Cu at (187.3, 60.4)
- added C19: 100n, Capacitor_SMD:C_0402_1005Metric, F.Cu at (192.0, 64.8)
- added C20: 10n, Capacitor_SMD:C_0402_1005Metric, F.Cu at (150.5, 106.0)
- added C21: 22p, Capacitor_SMD:C_0402_1005Metric, F.Cu at (147.0, 102.6)
- added C22: 22p, Capacitor_SMD:C_0402_1005Metric, F.Cu at (147.0, 110.6)
- added C23: 10u, Capacitor_SMD:C_0603_1608Metric, F.Cu at (171.0, 116.0)
- added C24: 100n, Capacitor_SMD:C_0402_1005Metric, F.Cu at (164.5, 114.0)
- added C25: 1u, Capacitor_SMD:C_0402_1005Metric, F.Cu at (161.5, 114.0)
- added C26: 100n, Capacitor_SMD:C_0402_1005Metric, F.Cu at (161.3, 111.0)
- added C27: 100n, Capacitor_SMD:C_0402_1005Metric, F.Cu at (158.5, 111.0)
- added C28: 100n, Capacitor_SMD:C_0402_1005Metric, F.Cu at (164.5, 116.0)
- added C29: 100n, Capacitor_SMD:C_0402_1005Metric, F.Cu at (161.5, 116.0)
- added C30: 100n, Capacitor_SMD:C_0402_1005Metric, F.Cu at (164.5, 111.0)
- added C31: 10n, Capacitor_SMD:C_0402_1005Metric, F.Cu at (153.0, 91.5)
- added C32: 100n, Capacitor_SMD:C_0402_1005Metric, F.Cu at (158.5, 114.0)
- added C38: 10n, Capacitor_SMD:C_0402_1005Metric, F.Cu at (149.0, 94.0)
- added C39: 10n, Capacitor_SMD:C_0402_1005Metric, F.Cu at (153.0, 88.5)
- added C5: 4.7n, Capacitor_SMD:C_0402_1005Metric, F.Cu at (193.0, 67.2)
- added C6: 4.7n, Capacitor_SMD:C_0402_1005Metric, F.Cu at (148.5, 102.5)
- added C7: 4.7n, Capacitor_SMD:C_0402_1005Metric, F.Cu at (196.0, 71.8)
- added C8: 1.5m, Capacitor_THT:CP_Radial_D35.0mm_P10.00mm_SnapIn, F.Cu at (116.0, 97.0)
- added C9: 1.5m, Capacitor_THT:CP_Radial_D35.0mm_P10.00mm_SnapIn, F.Cu at (116.0, 59.0)
- added D1: Red LED, LED_SMD:LED_0603_1608Metric, F.Cu at (169.0, 78.0)
- added D10: Blue LED, LED_SMD:LED_0603_1608Metric, F.Cu at (167.8, 86.0)
- added D11: Blue LED, LED_SMD:LED_0603_1608Metric, F.Cu at (170.4, 86.0)
- added D12: Blue LED, LED_SMD:LED_0603_1608Metric, F.Cu at (173.0, 86.0)
- added D2: Red LED, LED_SMD:LED_0603_1608Metric, F.Cu at (183.0, 75.4)
- added D3: Red LED, LED_SMD:LED_0603_1608Metric, F.Cu at (179.8, 75.4)
- added D4: Red LED, LED_SMD:LED_0603_1608Metric, F.Cu at (155.0, 107.8)
- added D5: Red LED, LED_SMD:LED_0603_1608Metric, F.Cu at (167.0, 106.0)
- added D6: Red LED, LED_SMD:LED_0603_1608Metric, F.Cu at (190.7, 107.5)
- added D7: Red LED, LED_SMD:LED_0603_1608Metric, F.Cu at (171.0, 103.0)
- added D8: Red LED, LED_SMD:LED_0603_1608Metric, F.Cu at (174.2, 117.0)
- added D9: Blue LED, LED_SMD:LED_0603_1608Metric, F.Cu at (165.2, 86.0)
- added H109: MountingHole_Pad, MountingHole:MountingHole_3.2mm_M3_Pad_Via, F.Cu at (200.0, 43.0)
- added H110: MountingHole_Pad, MountingHole:MountingHole_3.2mm_M3_Pad_Via, F.Cu at (102.7, 42.3)
- added H111: MountingHole_Pad, MountingHole:MountingHole_3.2mm_M3_Pad_Via, F.Cu at (198.0, 149.6)
- added H112: MountingHole_Pad, MountingHole:MountingHole_3.2mm_M3_Pad_Via, F.Cu at (102.3, 150.3)
- added H113: MountingHole_Pad, MountingHole:MountingHole_3.2mm_M3_Pad_Via, F.Cu at (141.0, 42.6)
- added H114: MountingHole_Pad, MountingHole:MountingHole_3.2mm_M3_Pad_Via, F.Cu at (140.0, 149.6)
- added J1: Conn_02x02_Top_Bottom, Connector_Molex:Molex_Micro-Fit_3.0_43045-0400_2x02_P3.00mm_Horizontal, F.Cu at (192.7, 113.5)
- added J4: Conn_01x02, Connector_JST:JST_XH_B2B-XH-A_1x02_P2.50mm_Vertical, F.Cu at (200.0, 87.0)
- added J5: Conn_01x02, Connector_JST:JST_XH_B2B-XH-A_1x02_P2.50mm_Vertical, F.Cu at (200.0, 97.0)
- added J6: Conn_ST_STDC14, Connector_PinHeader_1.27mm:PinHeader_2x07_P1.27mm_Vertical_SMD, F.Cu at (157.8, 80.2)
- added L1: 39n, Inductor_SMD:L_0603_1608Metric, F.Cu at (158.5, 116.0)
- added Q5: SQ2310ES, Package_TO_SOT_SMD:SOT-23, F.Cu at (185.5, 89.5)
- added R1: 390, Resistor_SMD:R_0402_1005Metric, F.Cu at (165.5, 77.0)
- added R10: 390, Resistor_SMD:R_0402_1005Metric, F.Cu at (174.4, 114.0)
- added R11: 22, Resistor_SMD:R_0402_1005Metric, F.Cu at (166.0, 91.0)
- added R12: 10k, Resistor_SMD:R_0402_1005Metric, F.Cu at (169.0, 91.5)
- added R1201: 200, Resistor_SMD:R_0402_1005Metric, F.Cu at (181.0, 97.0)
- added R15: 10k, Resistor_SMD:R_0402_1005Metric, F.Cu at (150.0, 88.5)
- added R18: 390, Resistor_SMD:R_0402_1005Metric, F.Cu at (166.6, 80.7)
- added R19: 390, Resistor_SMD:R_0402_1005Metric, F.Cu at (168.6, 80.7)
- added R2: 10k, Resistor_SMD:R_0402_1005Metric, F.Cu at (182.8, 80.4)
- added R20: 390, Resistor_SMD:R_0402_1005Metric, F.Cu at (170.6, 80.7)
- added R21: 390, Resistor_SMD:R_0402_1005Metric, F.Cu at (172.6, 80.7)
- added R3: 100k, Resistor_SMD:R_0402_1005Metric, F.Cu at (178.5, 70.5)
- added R4: 390, Resistor_SMD:R_0402_1005Metric, F.Cu at (155.0, 111.0)
- added R5: 8.2K, Resistor_SMD:R_0402_1005Metric, F.Cu at (175.8, 70.5)
- added R6: 2k7, Resistor_SMD:R_0402_1005Metric, F.Cu at (179.8, 80.4)
- added R7: 390, Resistor_SMD:R_0402_1005Metric, F.Cu at (166.5, 108.5)
- added R8: 390, Resistor_SMD:R_0402_1005Metric, F.Cu at (171.0, 107.0)
- added R9: 680, Resistor_SMD:R_0402_1005Metric, F.Cu at (191.0, 90.5)
- added SW1: SW_Push, Custom:435451019820, F.Cu at (200.9, 64.7)
- added SW2: SW_Push, Custom:435451019820, F.Cu at (200.9, 68.5)
- added SW7: SW_Push, Custom:435451019820, F.Cu at (200.9, 72.3)
- added SW8: SW_Push, Custom:435451019820, F.Cu at (200.9, 76.2)
- added U1201: TCN75A, Package_SO:SOIC-8_3.9x4.9mm_P1.27mm, F.Cu at (173.5, 98.1)
- added U2: GO 10-SME/SP3, Custom:SOIC8-GO-SME&slash_SP3_LEM, F.Cu at (184.0, 69.5)
- added U4: AZ1117-3.3, Package_TO_SOT_SMD:SOT-223-3_TabPin2, F.Cu at (181.8, 104.5)
- added U5: MAX3097ECSE+, Package_SO:SOIC-16_3.9x9.9mm_P1.27mm, F.Cu at (143.5, 94.6)
- added U6: STM32G474RETx, Package_QFP:LQFP-64_10x10mm_P0.5mm, F.Cu at (158.8, 99.0)
- added Y1: 16M, Custom:ABLS-7.3728MHZ-CL-RESR-A-1-G-F, F.Cu at (142.0, 107.3)
Routing:
- net +3.3V: track 0.00 -> 67.6 mm, vias 0 -> 1
- net GND: track 0.00 -> 61.0 mm, vias 0 -> 8
- net (no net): track 0.00 -> 19.8 mm, vias 0 -> 1
- net Net-(J4-Pin_2): track 0.00 -> 15.6 mm
- net /In_B_H: track 0.00 -> 7.64 mm
- net /MCU_STM32G475/USR_BTN_2: track 0.00 -> 6.45 mm
- net /Imes_vbus: track 0.00 -> 2.78 mm
- net /Uref_vbus: track 0.00 -> 2.77 mm
- net /In_A_L: track 0.00 -> 2.33 mm
- net Net-(D4-K): track 0.00 -> 1.91 mm
- net +5V: vias 0 -> 1
- added copper zone on In2.Cu, net +3.3V
- added copper zone on In2.Cu, net +5V
- added copper zone on B.Cu, net GND
- added copper zone on F.Cu, net GND
- added copper zone on In1.Cu, net GND
Other:
- board outline added: 107 x 119 mm

Commit message: almost finished pcb
Parts:
- removed D2: Red LED, LED_SMD:LED_0603_1608Metric
- removed R2: 10k, Resistor_SMD:R_0402_1005Metric
- added BT1: Battery, Connector_AMASS:AMASS_XT60-F_1x02_P7.20mm_Vertical, F.Cu at (136.8, 161.0)
- added C1: 10u, Capacitor_SMD:C_0603_1608Metric_Pad1.08x0.95mm_HandSolder, F.Cu at (191.2, 150.4)
- added C2: 1u, Capacitor_SMD:C_0603_1608Metric_Pad1.08x0.95mm_HandSolder, B.Cu at (177.1, 123.4)
- added C3: 1u, Capacitor_SMD:C_0603_1608Metric_Pad1.08x0.95mm_HandSolder, B.Cu at (182.7, 114.7)
- added C33: 10u, Capacitor_SMD:C_0603_1608Metric_Pad1.08x0.95mm_HandSolder, F.Cu at (160.8, 139.9)
- added C34: 4.7nF, Capacitor_SMD:C_0402_1005Metric_Pad0.74x0.62mm_HandSolder, F.Cu at (155.6, 135.1)
- added C35: 22nF, Capacitor_SMD:C_0402_1005Metric, F.Cu at (150.9, 134.3)
- added C36: 47u, Capacitor_SMD:C_0805_2012Metric, F.Cu at (149.1, 131.2)
- added C4: 10u, Capacitor_SMD:C_0603_1608Metric_Pad1.08x0.95mm_HandSolder, F.Cu at (175.4, 143.3)
- added Converter_DCDC_WPMDH1302401: ~, Package_TO_SOT_SMD:TO-263-7_TabPin8, F.Cu at (154.0, 146.5)
- added J2: 173010542, Connector_PinHeader_2.54mm:PinHeader_1x03_P2.54mm_Vertical, F.Cu at (150.2, 123.2)
- added J3: Conn_02x05_Odd_Even, Connector_PinHeader_2.54mm:PinHeader_2x05_P2.54mm_Vertical, F.Cu at (157.0, 95.4)
- added R13: 10k, Resistor_SMD:R_0402_1005Metric, F.Cu at (181.9, 61.3)
- added R14: 10k, Resistor_SMD:R_0402_1005Metric, F.Cu at (172.5, 60.9)
- added R16: 10k, Resistor_SMD:R_0402_1005Metric, F.Cu at (182.0, 65.2)
- added R17: 10k, Resistor_SMD:R_0402_1005Metric, F.Cu at (172.5, 64.8)
- added R22: 10k, Resistor_SMD:R_0402_1005Metric, F.Cu at (182.2, 69.1)
- added R23: 10k, Resistor_SMD:R_0402_1005Metric, F.Cu at (172.5, 68.6)
- added R24: 10k, Resistor_SMD:R_0402_1005Metric, F.Cu at (182.1, 73.0)
- added R25: 10k, Resistor_SMD:R_0402_1005Metric, F.Cu at (172.5, 72.5)
- added R26: 287k, Resistor_SMD:R_0402_1005Metric, F.Cu at (158.8, 135.1)
- added R27: 1.91k, Resistor_SMD:R_0402_1005Metric, F.Cu at (153.5, 133.1)
- added R28: 34k, Resistor_SMD:R_0402_1005Metric, F.Cu at (150.9, 133.1)
- added TP1: TestPoint, TestPoint:TestPoint_Pad_D2.0mm, F.Cu at (146.0, 140.0)
- added TP2: TestPoint, TestPoint:TestPoint_Pad_D2.0mm, F.Cu at (150.2, 128.3)
- added TP3: TestPoint, TestPoint:TestPoint_Pad_D2.0mm, F.Cu at (159.2, 123.6)
- added TP4: TestPoint, TestPoint:TestPoint_Pad_D2.0mm, F.Cu at (168.4, 110.0)
- added U1: MIC4606, Package_SO:TSSOP-16-1EP_4.4x5mm_P0.65mm_EP3x3mm, B.Cu at (179.1, 116.7)
- added U3: GO 10-SME/SP3, Custom:SOIC8-GO-SME&slash_SP3_LEM, F.Cu at (184.5, 158.6)
- added U7: CSD86350Q5D, CSD87351Q5D:DQY0008A, F.Cu at (186.4, 148.2)
- added U8: CSD86350Q5D, CSD87351Q5D:DQY0008A, F.Cu at (173.1, 147.6)
- C1201, U1201: moved to B.Cu
- C17: footprint Capacitor_SMD:CP_Elec_4x5.4 -> Capacitor_SMD:C_0603_1608Metric_Pad1.08x0.95mm_HandSolder
- C18: footprint Capacitor_SMD:CP_Elec_5x5.4 -> Capacitor_SMD:C_0603_1608Metric_Pad1.08x0.95mm_HandSolder
- C23: footprint Capacitor_SMD:C_0603_1608Metric -> Capacitor_SMD:C_0603_1608Metric_Pad1.08x0.95mm_HandSolder
- C25: footprint Capacitor_SMD:C_0402_1005Metric -> Capacitor_SMD:C_0603_1608Metric_Pad1.08x0.95mm_HandSolder
- moved C13 96.7 mm to (137.5, 146.8), turned to -90 degrees
- moved U2 90.4 mm to (141.1, 149.0), turned to 90 degrees
- moved C14 89.2 mm to (140.7, 143.9), turned to 90 degrees
- moved C7 88.8 mm to (189.2, 160.3), turned to -90 degrees
- moved C5 88.0 mm to (186.8, 154.9), turned to 180 degrees
- moved C15 87.6 mm to (142.5, 144.6)
- moved R5 77.4 mm to (200.3, 143.9), turned to 0 degrees
- moved R3 74.6 mm to (199.3, 142.2), turned to 0 degrees
- moved C6 68.5 mm to (189.3, 157.5), turned to 90 degrees
- moved R9 57.6 mm to (209.0, 145.2)
- moved D3 57.2 mm to (172.8, 132.2)
- moved C18 57.0 mm to (169.1, 114.4)
- moved C20 55.1 mm to (183.4, 61.8), turned to 180 degrees
- moved R11 54.0 mm to (204.7, 128.6)
- moved J6 53.4 mm to (204.6, 105.8)
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Routing:
- net +3.3V: track 67.6 -> 120.3 mm, vias 1 -> 13
- net VBUS: track 0.00 -> 48.1 mm, vias 0 -> 15
- net GND: track 61.0 -> 13.0 mm, vias 8 -> 6
- net /MCU_STM32G475/SWCLK: track 0.00 -> 46.7 mm
- net /MCU_STM32G475/SWDIO: track 0.00 -> 42.9 mm
- net //B: track 0.00 -> 33.0 mm
- net /MCU_STM32G475/USR_LED_4: track 0.00 -> 29.2 mm
- net /MCU_STM32G475/USR_LED_3: track 0.00 -> 28.4 mm
- net /MCU_STM32G475/USR_LED_2: track 0.00 -> 27.5 mm
- net /MCU_STM32G475/USR_LED_1: track 0.00 -> 26.7 mm
- net //A: track 0.00 -> 24.5 mm
- net Net-(U6-PF0): track 0.00 -> 20.5 mm
- net (no net): track 19.8 -> 0.00 mm
- net /MCU_STM32G475/VCP_RX: track 0.00 -> 17.9 mm
- net /MCU_STM32G475/VCP_TX: track 0.00 -> 17.8 mm
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- added copper zone on In2.Cu, net VBUS
Other:
- board size 107 x 119 mm -> 120 x 120 mm
- board text removed: "AAP_Inverter v1 07/09/23 N. PAPAZOGLOU A. MARTIN P. TOUSSAINT"
- board text removed: "U"
- board text removed: "V"
- board text removed: "W"
- board text removed: "Warning 230V AC AREA"

Commit message: finalization
Rooting and last edits ready to go
Parts:
- removed Converter_DCDC_WPMDH1302401: ~, Package_TO_SOT_SMD:TO-263-7_TabPin8
- removed G***: LOGO, LOGO
- removed H110, H112: MountingHole_Pad, MountingHole:MountingHole_3.2mm_M3_Pad_Via
- removed TP2, TP3: TestPoint, TestPoint:TestPoint_Pad_D2.0mm
- added J7: Conn_01x02, Connector_JST:JST_XH_B2B-XH-A_1x02_P2.50mm_Vertical, F.Cu at (207.5, 121.0)
- added TP 5V: TestPoint, TestPoint:TestPoint_Pad_D2.0mm, F.Cu at (166.7, 126.6)
- added TP 7.5V: TestPoint, TestPoint:TestPoint_Pad_D2.0mm, F.Cu at (157.1, 131.2)
- added WPMDH1302401: ~, Package_TO_SOT_SMD:TO-263-7_TabPin8, F.Cu at (162.8, 149.9)
- C10, C11, C12, C8, C9: value 1.5m -> 220u; footprint Capacitor_THT:CP_Radial_D35.0mm_P10.00mm_SnapIn -> Capacitor_SMD:CP_Elec_10x10.5
- R1201: moved to B.Cu
- TP 3.3V: renamed from TP4
- moved J3 69.9 mm to (167.5, 164.5), turned to 90 degrees
- moved C9 69.2 mm to (147.0, 132.5), turned to -90 degrees
- moved C12 68.5 mm to (155.5, 72.5)
- moved R23 48.1 mm to (198.1, 109.3)
- moved R22 47.7 mm to (207.1, 109.8)
- moved C38 47.7 mm to (209.2, 110.3)
- moved SW7 47.7 mm to (202.3, 110.1)
- moved C10 46.9 mm to (147.0, 152.0), turned to -90 degrees
- moved BT1 45.7 mm to (147.5, 116.6), turned to 90 degrees
- moved D6 44.8 mm to (171.5, 132.7), turned to 90 degrees
- moved C13 42.4 mm to (159.2, 110.4), turned to 180 degrees
- moved R9 38.7 mm to (171.5, 135.6)
- moved U2 38.4 mm to (157.0, 114.0), turned to 0 degrees
- moved C14 37.3 mm to (162.1, 113.4), turned to 0 degrees
- moved C8 35.5 mm to (155.0, 98.5)
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Connections:
- U6 pad 22: unconnected-(U6-PC4-Pad22) -> /MCU_STM32G475/USART1_RX
- U6 pad 23: unconnected-(U6-PC5-Pad23) -> /MCU_STM32G475/USART1_TX
Routing:
- net /ARM_B: track 7.67 -> 76.1 mm, vias 0 -> 2
- net /Imes_mot: track 2.08 -> 63.4 mm, vias 0 -> 2
- net /PWM_FAN: track 0.00 -> 61.1 mm, vias 0 -> 2
- net /VBus_Sense: track 3.86 -> 60.9 mm, vias 0 -> 2
- net /A: track 7.91 -> 63.4 mm, vias 0 -> 1
- net /B: track 8.11 -> 61.8 mm, vias 0 -> 1
- net /Z: track 7.80 -> 61.2 mm, vias 0 -> 1
- net //Z: track 12.7 -> 64.4 mm, vias 0 -> 1
- net VBUS: track 48.1 -> 93.4 mm, vias 15 -> 36
- net /ARM_IN_A: track 11.2 -> 54.1 mm, vias 0 -> 1
- net +3.3V: track 120.3 -> 162.4 mm, vias 13 -> 19
- net //A: track 24.5 -> 65.6 mm, vias 0 -> 1
- net /MCU_STM32G475/NRST: track 3.25 -> 41.4 mm, vias 1 -> 2
- net /Cmd_L_B: track 0.00 -> 37.2 mm, vias 0 -> 1
- net /In_B_H: track 0.00 -> 36.8 mm, vias 0 -> 2
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- added copper zone on B.Cu, net (none)
- added copper zone on F.Cu, net (none)
Other:
- board size 120 x 120 mm -> 75 x 105 mm

Commit message: PCB motor oof
Parts:
- J7: value Conn_01x02 -> Conn_01x04_Pin; footprint Connector_JST:JST_XH_B2B-XH-A_1x02_P2.50mm_Vertical -> Connector_JST:JST_XH_B4B-XH-A_1x04_P2.50mm_Vertical
- TP4: renamed from TP 3.3V
- moved R22 2.73 mm to (204.3, 109.4)
- moved C38 2.73 mm to (206.4, 109.9)
- moved R23 2.73 mm to (195.4, 108.9)
- moved SW7 2.73 mm to (199.7, 109.7)
- moved J4 2.28 mm to (209.5, 130.6), turned to 180 degrees
- moved J5 2.12 mm to (209.5, 137.8), turned to 180 degrees
- moved J7 1.44 mm to (208.2, 122.2)
Connections:
- J7 pad 1: /MCU_STM32G475/USART1_RX -> unconnected-(J7-Pin_1-Pad1)
- J7 pad 2: /MCU_STM32G475/USART1_TX -> /MCU_STM32G475/USART1_RX
Routing:
- net Net-(J4-Pin_2): track 18.3 -> 16.4 mm
- net +3.3V: track 162.4 -> 161.4 mm, vias 19 -> 18
- net /MCU_STM32G475/USART1_TX: track 29.0 -> 29.9 mm

Commit message: hello
Parts:
- removed C11, C12: 220u, Capacitor_SMD:CP_Elec_10x10.5
- BT1: footprint Connector_AMASS:AMASS_XT60-F_1x02_P7.20mm_Vertical -> Connector_AMASS:AMASS_XT60-M_1x02_P7.20mm_Vertical
- C33, C34, C35, C36, R26, R27, R28, WPMDH1302401: moved to B.Cu
- moved D8 66.4 mm to (240.3, 122.3)
- moved R10 66.4 mm to (240.3, 125.4)
- moved D6 66.4 mm to (237.1, 122.3)
- moved R9 66.4 mm to (237.1, 125.2)
- moved D3 64.0 mm to (231.7, 121.6)
- moved R6 64.0 mm to (231.7, 124.5)
- moved WPMDH1302401 43.7 mm to (151.8, 107.5), turned to 90 degrees
- moved C10 43.2 mm to (169.0, 114.8), turned to 0 degrees
- moved TP4 34.1 mm to (198.6, 122.3)
- moved R5 31.5 mm to (189.0, 114.5)
- moved R3 31.1 mm to (188.0, 113.1)
- moved C33 31.0 mm to (158.7, 114.2), turned to 90 degrees
- moved H113 29.1 mm to (146.3, 86.8)
- moved J1 28.4 mm to (177.0, 136.5), turned to 180 degrees
- moved J3 25.7 mm to (156.1, 141.6)
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Routing:
- net +3.3V: track 161.4 -> 87.3 mm, vias 18 -> 17
- net //B: track 64.2 -> 6.86 mm
- net /ARM_B: track 76.1 -> 19.5 mm, vias 2 -> 8
- net //Z: track 64.4 -> 8.02 mm
- net /Z: track 61.2 -> 5.26 mm
- net /B: track 61.8 -> 7.51 mm
- net //A: track 65.6 -> 12.3 mm
- net /A: track 63.4 -> 11.2 mm
- net VBUS: track 93.4 -> 48.0 mm, vias 36 -> 39
- net /VBus_Sense: track 60.9 -> 22.7 mm
- net /ARM_IN_A: track 54.1 -> 21.1 mm, vias 1 -> 2
- net /Imes_mot: track 63.4 -> 41.1 mm
- net /Cmd_L_A: track 36.2 -> 14.4 mm
- net /Cmd_H_A: track 30.6 -> 9.05 mm
- net /Imes_vbus: track 37.7 -> 56.3 mm
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- added copper zone on B.Cu, net +7.5V
- added copper zone on F.Cu, net /ARM_B
- added copper zone on F.Cu, net /ARM_IN_A
- added copper zone on F.Cu, net /ARM_OUT_A
- added copper zone on F.Cu, net Net-(BT1-+)
- added copper zone on F.Cu, net VBUS
Other:
- board size 75 x 105 mm -> 70.1 x 105 mm

Commit message: yo
Parts:
- moved R6 47.6 mm to (184.2, 127.9)
- moved D3 47.6 mm to (184.3, 125.2)
- moved R10 42.7 mm to (198.4, 117.1), turned to 90 degrees
- moved D8 42.0 mm to (198.4, 120.2), turned to -90 degrees
- moved D6 29.8 mm to (208.0, 128.7)
- moved R9 29.8 mm to (208.0, 131.6)
- moved H109 14.2 mm to (214.3, 80.7)
- moved H113 5.36 mm to (151.6, 86.0)
- moved C1 4.82 mm to (182.7, 120.8)
- moved H111 3.30 mm to (202.7, 148.6)
- moved C4 1.92 mm to (173.4, 122.4)
- moved TP 5V 1.62 mm to (189.2, 127.5)
- moved H114 1.41 mm to (150.0, 149.0)
- moved U7 1.33 mm to (179.8, 126.9)
- moved TP4 1.21 mm to (198.7, 123.5)
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Routing:
- net //Z: track 8.02 -> 41.4 mm
- net //B: track 6.86 -> 40.0 mm
- net /Z: track 5.26 -> 38.0 mm
- net +3.3V: track 87.3 -> 118.7 mm, vias 17 -> 20
- net /B: track 7.51 -> 36.3 mm
- net //A: track 12.3 -> 38.6 mm
- net /A: track 11.2 -> 34.7 mm
- net /ARM_IN_A: track 21.1 -> 7.73 mm, vias 2 -> 6
- net /Cmd_L_A: track 14.4 -> 3.52 mm
- net /In_B_H: track 26.3 -> 34.5 mm
- net /In_B_L: track 23.7 -> 30.3 mm
- net /In_A_L: track 11.3 -> 15.9 mm
- net /In_A_H: track 10.9 -> 14.3 mm
- net Net-(J4-Pin_2): track 14.3 -> 17.5 mm
- net +5V: track 2.69 -> 3.80 mm, vias 3 -> 4
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Other:
- board text added: "RX"
- board text added: "TX"

Commit message: Done !
Parts:
- moved H109 10.2 mm to (205.0, 85.0)
- moved R19 8.75 mm to (195.5, 89.3)
- moved R18 8.64 mm to (195.5, 87.7)
- moved R20 8.58 mm to (195.6, 90.9)
- moved D10 8.17 mm to (192.4, 89.3)
- moved D11 8.15 mm to (192.4, 90.9)
- moved D9 8.14 mm to (192.4, 87.7)
- moved H113 6.68 mm to (145.0, 85.0)
- moved H114 6.40 mm to (145.0, 145.0)
- moved H111 4.27 mm to (205.0, 145.0)
- moved TP 7.5V 3.23 mm to (166.6, 135.4)
- moved U2 2.90 mm to (143.7, 119.5)
- moved C13 2.80 mm to (141.7, 114.6)
- moved C14 2.80 mm to (143.1, 114.5)
- moved C15 2.80 mm to (145.1, 115.1)
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Routing:
- net VBUS: track 49.0 -> 27.9 mm, vias 39 -> 50
- net +7.5V: track 30.7 -> 51.8 mm, vias 3 -> 2
- net /ARM_IN_A: track 7.73 -> 21.8 mm, vias 6 -> 1
- net /ARM_B: track 18.6 -> 29.5 mm, vias 8 -> 2
- net /Cmd_L_A: track 3.52 -> 14.2 mm
- net /MCU_STM32G475/USR_LED_1: track 18.8 -> 9.56 mm
- net +3.3V: track 118.7 -> 127.6 mm, vias 20 -> 19
- net /MCU_STM32G475/USR_LED_2: track 17.0 -> 8.31 mm
- net /MCU_STM32G475/USR_LED_3: track 15.7 -> 7.08 mm
- net GND: track 22.9 -> 30.1 mm, vias 86 -> 68
- net /MCU_STM32G475/USR_BTN_1: track 20.8 -> 18.9 mm
- net Net-(Converter_DCDC_WPMDH1302401-RON): track 5.32 -> 3.52 mm
- net Net-(D6-K): track 0.00 -> 1.60 mm
- net /Imes_vbus: track 56.3 -> 55.2 mm
- net Net-(D10-K): track 2.40 -> 1.81 mm
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Other:
- board size 70.1 x 105 mm -> 70 x 70 mm
