File: Hardware/Hardware_électronique/MainBoard/PCB_test/MainBoard_test1/Rpi.kicad_sch (KiCad schematic)
At the start: 1 part, among them J1 Conn_02x20_Odd_Even

Commit message: PCB motor oof
Connections:
- net GND: now reaches J1.14 (Pin_14)
- net GND: now also J1.6 (Pin_6), J1.9 (Pin_9)
- net 5V: now reaches J1.2 (Pin_2)
- net 5V: now also J1.4 (Pin_4)
- no-connect marks 12 -> 7
