File: Hardware/Hardware_électronique/MainBoard/PCB_test/MainBoard_test1/_autosave-test1.kicad_sch (KiCad schematic)
At the start: 2 parts

Commit message: PCB motor oof
Other:
- removed sheet Buck7
Changed lines of the file:
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@@
-	)
-	(sheet
-		(at 31.75 115.57)
-		(size 17.78 5.5)
-		(fields_autoplaced yes)
-		(stroke
-			(width 0.1524)
-			(type solid)
-		)
-		(fill
-			(color 0 0 0 0.0000)
-		)
-		(property "Sheetname" "Buck7"
-			(at 31.75 114.8584 0)
-			(effects
-				(font
-					(size 1.27 1.27)
-				)
-				(justify left bottom)
-			)
-		)
-		(property "Sheetfile" "buck7.4V.kicad_sch"
-			(at 31.75 121.6546 0)
-			(effects
-				(font
-					(size 1.27 1.27)
-				)
-				(justify left top)
-			)
-		)
-		(pin "Vin" input
-			(at 31.75 118.13 180)
-			(effects
-				(font
-					(size 1.27 1.27)
-				)
-				(justify left)
-			)
-		)
-		(pin "Vout" output
-			(at 49.53 118.13 0)
-			(effects
-				(font
-					(size 1.27 1.27)
-				)
-				(justify right)
-			)
-		)
-		(instances
-			(project "test1"
-				(path "/6efb9aa2-c304-47cb-bf47-2a5d20e826bc"
-					(page "4")
-				)
-			)
-		)
 	)
 	(sheet
