File: Hardware/Hardware_électronique/MainBoard/PCB_test/MainBoard_test1/conn_ext.kicad_sch (KiCad schematic)
At the start: 18 parts

Commit message: commitment
Parts:
- removed D1, D2, D3, D4, D5, D6, D7, D8, D9: ESD7C5.0DT5G, Package_TO_SOT_SMD:SOT-416, symbol Power_Protection:RCLAMP0582B
- removed LIDAR1, UART1, UART2, UART3, UART4, UART5, UART6, UART7, UART8: Conn_01x04_Male, Connector_JST:JST_XH_B4B-XH-A_1x04_P2.50mm_Vertical, symbol Connector:Conn_01x04_Male
