File: Hardware/Hardware_électronique/MainBoard/PCB_test/MainBoard_test1/buck5V.kicad_sch (KiCad schematic)
At the start: 11 parts, among them U3 LT1076CR-PBF

Commit message: PCB motor oof
Changed lines of the file:
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@@
 	)
 	(hierarchical_label "Vout"
-		(shape input)
+		(shape output)
 		(at 123.19 101.6 90)
 		(fields_autoplaced yes)
@@
 	)
 	(hierarchical_label "Vout"
-		(shape input)
+		(shape output)
 		(at 149.86 63.5 0)
 		(fields_autoplaced yes)

Commit message: hey
Parts:
- added C48: C_Small, symbol Device:C_Small
- added U5: ~, symbol Custom:LM53603AMPWPT
Changed lines of the file:
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@@
+	)
+	(symbol
+		(lib_id "Device:C_Small")
+		(at 154.94 83.82 0)
+		(unit 1)
+		(exclude_from_sim no)
+		(in_bom yes)
+		(on_board yes)
+		(dnp no)
+		(fields_autoplaced yes)
+		(property "Reference" "C48"
+			(at 157.48 82.5562 0)
+			(effects
+				(font
+					(size 1.27 1.27)
+				)
+				(justify left)
+			)
+		)
+		(property "Value" "C_Small"
+			(at 157.48 85.0962 0)
+			(effects
+				(font
+					(size 1.27 1.27)
+				)
+				(justify left)
+			)
+		)
+		(property "Footprint" ""
+			(at 154.94 83.82 0)
+			(effects
+				(font
+					(size 1.27 1.27)
+				)
+				(hide yes)
+			)
+		)
+		(property "Datasheet" "~"
+			(at 154.94 83.82 0)
+			(effects
+				(font
+					(size 1.27 1.27)
+				)
+				(hide yes)
+			)
+		)
+		(property "Description" "Unpolarized capacitor, small symbol"
+			(at 154.94 83.82 0)
+			(effects
+				(font
+					(size 1.27 1.27)
+				)
+				(hide yes)
+			)
+		)
+		(pin "1"
+		)
+		(pin "2"
+		)
+		(instances
+			(project ""
+				(path "/6efb9aa2-c304-47cb-bf47-2a5d20e826bc/26d4398e-0944-4bb2-b6fd-d788547aa7d2"
+					(reference "C48")
+					(unit 1)
+				)
+			)
+		)
 	)
 	(symbol
@@
 			)
 		)
-		(property "Datasheet" "https://www.mouser.fr/datasheet/2/240/media-3323546.pdf"
+		(property "Datasheet" "https://www.mouser.fr/ProductDetail/ROHM-Semiconductor/RSX301L-30DDTE25?qs=sGAEpiMZZMtbRapU8LlZD%252B6h%2FWulpAkr%2FY1xa87RQph8xMmqFKqxyQ%3D%3D"
 			(at 116.84 68.58 0)
 			(effects
@@
 					(unit 1)
 				)
+			)
+		)
+	)
+	(symbol
+		(lib_id "Custom:LM53603AMPWPT")
+		(at 99.06 36.83 0)
+		(unit 1)
+		(exclude_from_sim no)
+		(in_bom yes)
+		(on_board yes)
+		(dnp no)
+		(fields_autoplaced yes)
+		(property "Reference" "U5"
+			(at 99.06 26.67 0)
+			(effects
+				(font
+					(size 1.27 1.27)
+				)
+			)
+		)
+		(property "Value" "~"
+			(at 99.06 29.21 0)
+			(effects
+				(font
+					(size 1.27 1.27)
+				)
+			)
+		)
+		(property "Footprint" ""
+			(at 99.06 36.83 0)
+			(effects
+				(font
+					(size 1.27 1.27)
+				)
+				(hide yes)
+			)
+		)
+		(property "Datasheet" ""
+			(at 99.06 36.83 0)
+			(effects
+				(font
+					(size 1.27 1.27)
+				)
+				(hide yes)
+			)
+		)
+		(property "Description" ""
+			(at 99.06 36.83 0)
+			(effects
+				(font
+					(size 1.27 1.27)
+				)
+				(hide yes)
+			)
+		)
+		(pin ""
+		)
+		(pin ""
+		)
+		(pin ""
+		)
+		(pin ""
+		)
+		(pin ""
+		)
+		(pin ""
+		)
+		(pin ""
+		)
+		(pin ""
+		)
+		(pin ""
+		)
+		(pin ""
+		)
+		(pin ""
+		)
+		(pin ""
+		)
+		(instances
+			(project ""
+				(path "/6efb9aa2-c304-47cb-bf47-2a5d20e826bc/26d4398e-0944-4bb2-b6fd-d788547aa7d2"
+					(reference "U5")
+					(unit 1)
+				)
