File: Hardware/Hardware_électronique/MainBoard/PCB_test/MainBoard_test1/test1.kicad_pcb (KiCad board)
At the start: 4 copper layers, 130 x 130 mm, 48 parts, among them J1 Conn_02x20_Odd_Even, J2 2309409-2, U1 STM32H735IGTx, U2 LT1076CR-PBF, U3 LT1076CR-PBF

Commit message: approaching end of schematics
Parts:
- removed ARU1, BAT1, BAT2: 180G-2, MainBoard:180G-2
- added ARU2: 180G-2, MainBoard:180G-2, F.Cu at (97.5, 79.7)
- added BT1: Battery, Connector_AMASS:AMASS_XT60PW-F_1x02_P7.20mm_Horizontal, F.Cu at (105.2, 54.6)
- added C30: 10n, Capacitor_SMD:C_0402_1005Metric, F.Cu at (56.7, 67.6)
- added C31: 10n, Capacitor_SMD:C_0402_1005Metric, F.Cu at (56.7, 69.6)
- added C32: 10n, Capacitor_SMD:C_0402_1005Metric, F.Cu at (56.7, 71.5)
- added C33: 10n, Capacitor_SMD:C_0402_1005Metric, F.Cu at (56.7, 73.5)
- added C34: 1u, Capacitor_SMD:C_0603_1608Metric_Pad1.08x0.95mm_HandSolder, F.Cu at (60.3, 67.9)
- added C35: 100n, Capacitor_SMD:C_0402_1005Metric, F.Cu at (56.7, 75.5)
- added C36: 100n, Capacitor_SMD:C_0402_1005Metric, F.Cu at (56.7, 77.5)
- added C37: 10u, Capacitor_SMD:C_0603_1608Metric_Pad1.08x0.95mm_HandSolder, F.Cu at (60.3, 70.4)
- added C38: 22u, Capacitor_SMD:C_0603_1608Metric_Pad1.08x0.95mm_HandSolder, F.Cu at (60.3, 72.9)
- added C39: 100n, Capacitor_SMD:C_0402_1005Metric, F.Cu at (56.7, 79.4)
- added C41: 100n, Capacitor_SMD:C_0402_1005Metric, F.Cu at (56.7, 81.4)
- added C45: 1u, Capacitor_SMD:C_0603_1608Metric_Pad1.08x0.95mm_HandSolder, F.Cu at (60.3, 75.4)
- added C46: 1u, Capacitor_SMD:C_0603_1608Metric_Pad1.08x0.95mm_HandSolder, F.Cu at (60.3, 77.9)
- added C47: 1u, Capacitor_SMD:C_0603_1608Metric_Pad1.08x0.95mm_HandSolder, F.Cu at (60.3, 80.4)
- added D14: LED, LED_SMD:LED_0603_1608Metric, F.Cu at (94.8, 61.5)
- added D15: LED, LED_SMD:LED_0603_1608Metric, F.Cu at (94.8, 64.1)
- added D16: LED, LED_SMD:LED_0603_1608Metric, F.Cu at (94.8, 66.7)
- added D17: LED, LED_SMD:LED_0603_1608Metric, F.Cu at (94.8, 69.3)
- added D18: Blue LED, LED_SMD:LED_0603_1608Metric, F.Cu at (57.3, 83.7)
- added D19: Blue LED, LED_SMD:LED_0603_1608Metric, F.Cu at (57.3, 86.3)
- added D20: Blue LED, LED_SMD:LED_0603_1608Metric, F.Cu at (57.3, 88.8)
- added D21: Blue LED, LED_SMD:LED_0603_1608Metric, F.Cu at (57.3, 91.4)
- added L3: 39n, Inductor_SMD:L_0603_1608Metric, F.Cu at (61.3, 92.0)
- added R10: 1k, Resistor_SMD:R_0402_1005Metric, F.Cu at (102.6, 86.7)
- added R11: 1k, Resistor_SMD:R_0402_1005Metric, F.Cu at (102.6, 88.7)
- added R12: 10k, Resistor_SMD:R_0402_1005Metric, F.Cu at (70.6, 83.4)
- added R13: 10k, Resistor_SMD:R_0402_1005Metric, F.Cu at (70.6, 85.4)
- added R14: 10k, Resistor_SMD:R_0402_1005Metric, F.Cu at (70.6, 87.3)
- added R15: 10k, Resistor_SMD:R_0402_1005Metric, F.Cu at (70.6, 89.3)
- added R16: 10k, Resistor_SMD:R_0402_1005Metric, F.Cu at (73.5, 83.4)
- added R17: 10k, Resistor_SMD:R_0402_1005Metric, F.Cu at (73.5, 85.4)
- added R18: 10k, Resistor_SMD:R_0402_1005Metric, F.Cu at (73.5, 87.3)
- added R19: 10k, Resistor_SMD:R_0402_1005Metric, F.Cu at (73.5, 89.3)
- added R20: 390, Resistor_SMD:R_0402_1005Metric, F.Cu at (76.4, 83.4)
- added R21: 390, Resistor_SMD:R_0402_1005Metric, F.Cu at (76.4, 85.4)
- added R22: 390, Resistor_SMD:R_0402_1005Metric, F.Cu at (76.4, 87.3)
- added R23: 390, Resistor_SMD:R_0402_1005Metric, F.Cu at (76.4, 89.3)
- added R8: 6k2, Resistor_SMD:R_0402_1005Metric, F.Cu at (102.6, 82.7)
- added R9: 1k8, Resistor_SMD:R_0402_1005Metric, F.Cu at (102.6, 84.7)
- added TP1: TestPoint, TestPoint:TestPoint_Pad_D2.0mm, F.Cu at (98.9, 59.7)
- added TP2: TestPoint, TestPoint:TestPoint_Pad_D2.0mm, F.Cu at (79.9, 84.4)
- added TP3: TestPoint, TestPoint:TestPoint_Pad_D2.0mm, F.Cu at (98.9, 63.7)
- added TP4: TestPoint, TestPoint:TestPoint_Pad_D2.0mm, F.Cu at (98.9, 67.8)
- added TP5: TestPoint, TestPoint:TestPoint_Pad_D2.0mm, F.Cu at (79.9, 88.5)
- added U4: AZ1117-3.3, Package_TO_SOT_SMD:SOT-223-3_TabPin2, F.Cu at (64.2, 86.6)
- J1: value Conn_02x20_Odd_Even -> Conn_RasPi
- J2: value 2309409-2 -> Conn_ST_STDC14; footprint footprints:CONN260_2309409-2_TEC -> Connector_PinHeader_1.27mm:PinHeader_2x07_P1.27mm_Vertical_SMD
- U1: moved to F.Cu
- moved C2 223.0 mm to (46.0, 126.8)
- moved U2 223.0 mm to (51.5, 116.6)
- moved C3 223.0 mm to (62.4, 129.7)
- moved C4 223.0 mm to (62.4, 131.7)
- moved C5 223.0 mm to (62.4, 113.3)
- moved C6 223.0 mm to (62.4, 119.2)
- moved L1 223.0 mm to (56.1, 127.6)
- moved R2 223.0 mm to (62.4, 123.8)
- moved R3 223.0 mm to (62.4, 125.7)
- moved R4 223.0 mm to (62.4, 127.7)
- moved LIDAR1 187.3 mm to (44.3, 41.6)
- moved UART3 167.4 mm to (44.3, 65.0), turned to 0 degrees
- moved D9 160.5 mm to (71.8, 75.0), turned to 0 degrees
- moved UART4 160.0 mm to (44.3, 72.8), turned to 0 degrees
- moved C10 149.2 mm to (107.2, 96.0)
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Connections:
- net /Buck7.4/Vout renamed +7.5V
- net /Buck7.4/vc renamed /Buck7.5/vc
- net /Buck7.4/voutbuck renamed /Buck7.5/voutbuck
- C10 pad 1: /Buck5.1/Vout -> +5V
- C11 pad 1: /Buck5.1/Vout -> +5V
- C2 pad 1: /Buck7.4/Vin -> VBUS
- C7 pad 1: /Buck5.1/Vin -> +BATT
- D1 pad 1: TX1 -> /STM32H735/TX1
- D1 pad 2: RX1 -> /STM32H735/RX1
- D11 pad 1: VBAT -> VBUS
- D2 pad 1: TX2 -> /STM32H735/TX3
- D2 pad 2: RX2 -> /STM32H735/RX3
- D3 pad 1: TX3 -> /STM32H735/TX4
- D3 pad 2: RX3 -> /STM32H735/RX4
- D4 pad 1: TX4 -> /STM32H735/TX5
- D4 pad 2: RX4 -> /STM32H735/RX5
- D5 pad 1: TX5 -> /STM32H735/TX2
- D5 pad 2: RX5 -> /STM32H735/RX2
- D6 pad 1: TX6 -> /STM32H735/TX6
- D6 pad 2: RX6 -> /STM32H735/RX6
- D7 pad 1: TX7 -> /STM32H735/TX7
- D7 pad 2: RX7 -> /STM32H735/RX7
- D8 pad 1: TX8 -> /STM32H735/TX8
- D8 pad 2: RX8 -> /STM32H735/RX8
- D9 pad 1: Lidar_TX -> /STM32H735/TX_Lidar
- D9 pad 2: Lidar_RX -> /STM32H735/RX_Lidar
- F1 pad 2: Net-(ARU1-Pad1) -> +BATT
- J1 pad 10: GPIO15_RXD -> /GPIO15_RXD
- J1 pad 11: GPIO17 -> unconnected-(J1-Pin_11-Pad11)
- J1 pad 12: GPIO18_PCMCLK -> unconnected-(J1-Pin_12-Pad12)
- J1 pad 13: GPIO27 -> unconnected-(J1-Pin_13-Pad13)
- J1 pad 14: unconnected-(J1-Pin_14-Pad14) -> GND
- J1 pad 15: GPIO22 -> unconnected-(J1-Pin_15-Pad15)
- J1 pad 16: GPIO23 -> unconnected-(J1-Pin_16-Pad16)
- J1 pad 18: GPIO24 -> unconnected-(J1-Pin_18-Pad18)
- J1 pad 19: GPIO10_MOSI -> unconnected-(J1-Pin_19-Pad19)
- J1 pad 2: unconnected-(J1-Pin_2-Pad2) -> +5V
- J1 pad 21: GPIO9_MISO -> unconnected-(J1-Pin_21-Pad21)
- J1 pad 22: GPIO25 -> unconnected-(J1-Pin_22-Pad22)
- J1 pad 23: GPIO11_SCLK -> unconnected-(J1-Pin_23-Pad23)
- J1 pad 24: GPIO8_CE0 -> unconnected-(J1-Pin_24-Pad24)
- J1 pad 26: GPIO7_CE1 -> unconnected-(J1-Pin_26-Pad26)
- J1 pad 27: GPIO0_ID_SD -> unconnected-(J1-Pin_27-Pad27)
- J1 pad 28: GPIO1_ID_SD -> unconnected-(J1-Pin_28-Pad28)
- J1 pad 29: GPIO5 -> unconnected-(J1-Pin_29-Pad29)
- J1 pad 3: GPIO2_SDA -> unconnected-(J1-Pin_3-Pad3)
- J1 pad 31: GPIO6 -> unconnected-(J1-Pin_31-Pad31)
- J1 pad 32: GPIO12_PWM0 -> unconnected-(J1-Pin_32-Pad32)
- J1 pad 33: GPIO13_PWM1 -> unconnected-(J1-Pin_33-Pad33)
- J1 pad 35: GPIO19_PCMFS -> unconnected-(J1-Pin_35-Pad35)
- J1 pad 36: GPIO16 -> unconnected-(J1-Pin_36-Pad36)
- J1 pad 37: GPIO26 -> unconnected-(J1-Pin_37-Pad37)
- J1 pad 38: GPIO20_PCMDIN -> unconnected-(J1-Pin_38-Pad38)
- J1 pad 4: unconnected-(J1-Pin_4-Pad4) -> +5V
- J1 pad 40: GPIO21_PCMDOUT -> unconnected-(J1-Pin_40-Pad40)
- J1 pad 5: GPIO3_SCL -> unconnected-(J1-Pin_5-Pad5)
- J1 pad 6: unconnected-(J1-Pin_6-Pad6) -> GND
- J1 pad 7: GPIO4_GPCLK0 -> unconnected-(J1-Pin_7-Pad7)
- J1 pad 8: GPIO14_TXD -> /GPIO14_TXD
- J1 pad 9: unconnected-(J1-Pin_9-Pad9) -> GND
- J2 pad 1: GND -> unconnected-(J2-NC-Pad1)
- J2 pad 11: unconnected-(J2-Pad11) -> GND
- J2 pad 12: unconnected-(J2-Pad12) -> /STM32H735/NRST
- J2 pad 13: unconnected-(J2-Pad13) -> /STM32H735/VCP_RX
- J2 pad 14: unconnected-(J2-Pad14) -> /STM32H735/VCP_TX
- J2 pad 3: unconnected-(J2-Pad3) -> +3.3V
- J2 pad 4: unconnected-(J2-Pad4) -> /STM32H735/SWDIO
- J2 pad 5: unconnected-(J2-Pad5) -> GND
- J2 pad 6: unconnected-(J2-Pad6) -> /STM32H735/SWCLK
- J2 pad 7: unconnected-(J2-Pad7) -> GND
- J2 pad 8: unconnected-(J2-Pad8) -> /STM32H735/SWO
- L2 pad 2: /Buck5.1/Vout -> +5V
- LIDAR1 pad 1: 5.1V -> VBUS
- LIDAR1 pad 2: Lidar_TX -> /STM32H735/TX_Lidar
- LIDAR1 pad 3: Lidar_RX -> /STM32H735/RX_Lidar
- R6 pad 1: /Buck5.1/Vout -> +5V
- U1 pad 1: unconnected-(U1-PE2-Pad1) -> /GPIO14_TXD
- U1 pad 100: Net-(U1-VSS-Pad100) -> GND
- U1 pad 101: unconnected-(U1-PJ8-Pad101) -> /STM32H735/TX8
- U1 pad 102: unconnected-(U1-PJ9-Pad102) -> /STM32H735/RX8
- U1 pad 105: unconnected-(U1-VDD-Pad105) -> +3.3V
- U1 pad 106: Net-(U1-VSS-Pad100) -> GND
- U1 pad 112: Net-(U1-VSS-Pad100) -> GND
- U1 pad 113: unconnected-(U1-VDD-Pad113) -> +3.3V
- U1 pad 119: Net-(U1-VSS-Pad100) -> GND
- U1 pad 12: Net-(U1-VSS-Pad100) -> GND
- U1 pad 120: unconnected-(U1-VDD50USB-Pad120) -> +5V
- U1 pad 121: unconnected-(U1-VDD33USB-Pad121) -> +3.3V
- U1 pad 122: unconnected-(U1-PC6-Pad122) -> /STM32H735/TX6
- U1 pad 123: unconnected-(U1-PC7-Pad123) -> /STM32H735/RX6
- U1 pad 126: unconnected-(U1-VDD-Pad126) -> +3.3V
- U1 pad 13: unconnected-(U1-VDD-Pad13) -> +3.3V
- U1 pad 130: unconnected-(U1-PA11-Pad130) -> /STM32H735/RX4
- U1 pad 131: unconnected-(U1-PA12-Pad131) -> /STM32H735/TX4
- U1 pad 132: unconnected-(U1-PA13(JTMS-Pad132) -> /STM32H735/SWDIO
- U1 pad 133: unconnected-(U1-VCAP-Pad133) -> Net-(C43-Pad1)
- U1 pad 134: Net-(U1-VSS-Pad100) -> GND
- U1 pad 135: unconnected-(U1-VDDLDO-Pad135) -> +3.3V
- U1 pad 136: unconnected-(U1-VDD-Pad136) -> +3.3V
- U1 pad 137: Net-(U1-VSS-Pad100) -> GND
- U1 pad 138: unconnected-(U1-PA14(JTCK-Pad138) -> /STM32H735/SWCLK
- U1 pad 14: unconnected-(U1-VSSSMPS-Pad14) -> GND
- U1 pad 148: unconnected-(U1-PD5-Pad148) -> /STM32H735/RX2
- U1 pad 149: unconnected-(U1-PD6-Pad149) -> /STM32H735/TX2
- U1 pad 151: Net-(U1-VSS-Pad100) -> GND
- U1 pad 152: unconnected-(U1-VDD-Pad152) -> +3.3V
- U1 pad 159: Net-(U1-VSS-Pad100) -> GND
- U1 pad 160: unconnected-(U1-VDD-Pad160) -> +3.3V
- U1 pad 162: unconnected-(U1-PB3(JTDO-Pad162) -> /STM32H735/SWO
- U1 pad 163: unconnected-(U1-PB4(NJTRST)-Pad163) -> /STM32H735/USR_BTN_1
- U1 pad 164: unconnected-(U1-PB5-Pad164) -> /STM32H735/USR_BTN_2
- U1 pad 167: unconnected-(U1-BOOT0-Pad167) -> /STM32H735/BOOT0
- U1 pad 172: unconnected-(U1-VCAP-Pad172) -> Net-(C44-Pad1)
- U1 pad 173: Net-(U1-VSS-Pad100) -> GND
- U1 pad 174: unconnected-(U1-PDR_ON-Pad174) -> GND
- U1 pad 175: unconnected-(U1-VDDLDO-Pad175) -> +3.3V
- U1 pad 176: unconnected-(U1-VDD-Pad176) -> +3.3V
- U1 pad 2: unconnected-(U1-PE3-Pad2) -> /GPIO15_RXD
- U1 pad 24: Net-(U1-VSS-Pad100) -> GND
- U1 pad 25: unconnected-(U1-VDD-Pad25) -> +3.3V
- U1 pad 33: unconnected-(U1-NRST-Pad33) -> /STM32H735/NRST
- U1 pad 38: unconnected-(U1-VSSA-Pad38) -> GND
- U1 pad 39: unconnected-(U1-VREF+-Pad39) -> +3.3VA
- U1 pad 40: unconnected-(U1-VDDA-Pad40) -> +3.3VA
- U1 pad 44: unconnected-(U1-VDD-Pad44) -> +3.3V
- U1 pad 45: Net-(U1-VSS-Pad100) -> GND
- U1 pad 47: Net-(U1-VSS-Pad100) -> GND
- U1 pad 48: unconnected-(U1-VDD-Pad48) -> +3.3V
- U1 pad 6: Net-(U1-VSS-Pad100) -> GND
- U1 pad 64: Net-(U1-VSS-Pad100) -> GND
- U1 pad 65: unconnected-(U1-VDD-Pad65) -> +3.3V
- U1 pad 67: unconnected-(U1-PE7-Pad67) -> /STM32H735/RX7
- U1 pad 68: unconnected-(U1-PE8-Pad68) -> /STM32H735/TX7
- U1 pad 7: unconnected-(U1-VDD-Pad7) -> +3.3V
- U1 pad 70: Net-(U1-VSS-Pad100) -> GND
- U1 pad 71: unconnected-(U1-VDD-Pad71) -> +3.3V
- U1 pad 78: unconnected-(U1-PB10-Pad78) -> /STM32H735/TX3
- U1 pad 79: unconnected-(U1-PB11-Pad79) -> /STM32H735/RX3
- U1 pad 8: unconnected-(U1-VBAT-Pad8) -> +3.3V
- U1 pad 80: unconnected-(U1-VCAP-Pad80) -> Net-(C42-Pad1)
- U1 pad 81: Net-(U1-VSS-Pad100) -> GND
- U1 pad 82: unconnected-(U1-VDDLDO-Pad82) -> +3.3V
- U1 pad 83: Net-(U1-VSS-Pad100) -> GND
- U1 pad 84: unconnected-(U1-VDD-Pad84) -> +3.3V
- U1 pad 85: unconnected-(U1-PB12-Pad85) -> /STM32H735/RX5
- U1 pad 86: unconnected-(U1-PB13-Pad86) -> /STM32H735/TX5
- U1 pad 87: unconnected-(U1-PB14-Pad87) -> /STM32H735/TX1
- U1 pad 88: unconnected-(U1-PB15-Pad88) -> /STM32H735/RX1
- U1 pad 92: unconnected-(U1-VDD-Pad92) -> +3.3V
- U1 pad 93: Net-(U1-VSS-Pad100) -> GND
- U1 pad 97: unconnected-(U1-PD14-Pad97) -> /STM32H735/RX_Lidar
- U1 pad 98: unconnected-(U1-PD15-Pad98) -> /STM32H735/TX_Lidar
- U1 pad 99: unconnected-(U1-VDD-Pad99) -> +3.3V
- U2 pad 1: /Buck7.4/Vin -> VBUS
- U2 pad 7: /Buck7.4/Vin -> VBUS
- U3 pad 1: /Buck5.1/Vin -> +BATT
- U3 pad 7: /Buck5.1/Vin -> +BATT
- UART1 pad 1: VBAT -> VBUS
- UART1 pad 2: TX1 -> /STM32H735/TX1
- UART1 pad 3: RX1 -> /STM32H735/RX1
- UART2 pad 1: VBAT -> VBUS
- UART2 pad 2: TX2 -> /STM32H735/TX3
- UART2 pad 3: RX2 -> /STM32H735/RX3
- UART3 pad 1: VBAT -> VBUS
- UART3 pad 2: TX3 -> /STM32H735/TX4
- UART3 pad 3: RX3 -> /STM32H735/RX4
- UART4 pad 1: VBAT -> VBUS
- UART4 pad 2: TX4 -> /STM32H735/TX5
- UART4 pad 3: RX4 -> /STM32H735/RX5
- UART5 pad 1: VBAT -> VBUS
- UART5 pad 2: TX5 -> /STM32H735/TX2
- UART5 pad 3: RX5 -> /STM32H735/RX2
- UART6 pad 1: VBAT -> VBUS
- UART6 pad 2: TX6 -> /STM32H735/TX6
- UART6 pad 3: RX6 -> /STM32H735/RX6
- UART7 pad 1: VBAT -> VBUS
- UART7 pad 2: TX7 -> /STM32H735/TX7
- UART7 pad 3: RX7 -> /STM32H735/RX7
- UART8 pad 1: VBAT -> VBUS
- UART8 pad 2: TX8 -> /STM32H735/TX8
- UART8 pad 3: RX8 -> /STM32H735/RX8
Routing:
- removed copper zone on B.Cu, net GND
- removed copper zone on F.Cu, net GND
Other:
- board outline removed
- copper layers 4 -> 2
