File: Hardware/Hardware_électronique/MainBoard/PCB_test/MainBoard_test1/test1.kicad_pcb (KiCad board)
At the start: 4 copper layers, 65 x 56 mm, 118 parts, among them J1 USB_C_Receptacle_USB2.0_16P, J2 Conn_ST_STDC14, J3 Conn_02x10_Odd_Even, Q1 PMOS, SW1 SW_Push, SW2 SW_Push, SW3 SW_Push, SW4 SW_Push, U1 STM32H735IGTx, U2 USBLC6-2SC6, U4 AZ1117-3.3

Commit message: Motherboard advance
Parts:
- C34, D1, D10, D11, D6, D7, D8, D9, F1, L3, Q1, R1, U3, U4: moved to B.Cu
- moved D10 97.6 mm to (59.7, 73.6), turned to 180 degrees
- moved Q1 96.3 mm to (53.9, 74.9)
- moved F1 93.4 mm to (52.5, 89.0), turned to 90 degrees
- moved U4 92.6 mm to (69.8, 70.5)
- moved U3 87.6 mm to (61.8, 78.8)
- moved D9 87.1 mm to (97.0, 63.9), turned to -90 degrees
- moved L3 85.6 mm to (93.6, 95.2)
- moved R1 83.0 mm to (53.9, 81.5)
- moved D1 82.0 mm to (106.3, 65.7)
- moved D11 79.4 mm to (53.7, 77.7), turned to 180 degrees
- moved D8 79.1 mm to (82.5, 64.6), turned to -90 degrees
- moved C23 77.1 mm to (88.4, 65.8)
- moved C22 75.4 mm to (91.0, 65.8), turned to 180 degrees
- moved C13 73.4 mm to (98.8, 66.0)
- moved BT1 72.5 mm to (48.1, 93.0)
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- renumbered UART3 to UART10, UART5 to UART2, UART2 to UART3, UART9 to UART4, UART4 to UART5
Routing:
- net /STM32H735/TX7: track 0.00 -> 36.2 mm
- net /STM32H735/RX7: track 0.00 -> 27.9 mm
- net /STM32H735/TX6: track 0.00 -> 25.2 mm
- net /STM32H735/TX3: track 0.00 -> 22.1 mm
- net /STM32H735/TX4: track 0.00 -> 21.9 mm
- net /STM32H735/TX8: track 0.00 -> 21.6 mm
- net /STM32H735/RX6: track 0.00 -> 21.2 mm
- net +3.3V: track 0.00 -> 20.8 mm, vias 0 -> 2
- net /STM32H735/RX3: track 0.00 -> 20.3 mm
- net /STM32H735/RX4: track 0.00 -> 20.0 mm
- net /STM32H735/RX8: track 0.00 -> 17.3 mm
- net /STM32H735/TX5: track 0.00 -> 16.3 mm
- net /STM32H735/RX1: track 0.00 -> 13.2 mm, vias 0 -> 1
- net /STM32H735/TX1: track 0.00 -> 11.8 mm, vias 0 -> 1
- net /STM32H735/RX5: track 0.00 -> 11.2 mm
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- added copper zone on In2.Cu, net +3.3V
- added copper zone on In2.Cu, net +5V
- added copper zone on B.Cu, net +BATT
- added copper zone on B.Cu, net Net-(ARU1-Pad1)
- added copper zone on B.Cu, net Net-(BT1-+)
- added copper zone on B.Cu, net VBUS
- added copper zone on F.Cu, net VBUS
- added copper zone on In2.Cu, net VBUS
Other:
- board size 65 x 56 mm -> 75 x 56 mm

Commit message: MotherBoard finished
Parts:
- removed D14, D16, D17: LED, LED_SMD:LED_0603_1608Metric
- removed R10, R11: 1k, Resistor_SMD:R_0402_1005Metric
- removed R8: 6k2, Resistor_SMD:R_0402_1005Metric
- removed TP2: TestPoint, TestPoint:TestPoint_Pad_D2.0mm
- C2, C7: footprint Capacitor_SMD:CP_Elec_4x5.4 -> Capacitor_SMD:C_0805_2012Metric; moved to B.Cu
- C3: footprint Capacitor_SMD:C_0805_2012Metric_Pad1.18x1.45mm_HandSolder -> Capacitor_SMD:C_0402_1005Metric_Pad0.74x0.62mm_HandSolder; moved to B.Cu
- C35, C36, C37, C38, C4, C5, C6, C8, D2, D22, D3, D4, D5, L1, R2, R3, R5, R6: moved to B.Cu
- C45, C46, C47: footprint Capacitor_SMD:C_0603_1608Metric_Pad1.08x0.95mm_HandSolder -> Capacitor_SMD:C_0402_1005Metric_Pad0.74x0.62mm_HandSolder
- USER BTN 1: renamed from SW2
- USER BTN2: renamed from SW3
- moved C7 115.9 mm to (56.0, 80.2), turned to -90 degrees
- moved C38 113.8 mm to (71.4, 65.8), turned to 180 degrees
- moved C2 110.5 mm to (58.3, 80.2), turned to -90 degrees
- moved C37 110.4 mm to (64.0, 67.1), turned to 90 degrees
- moved C47 97.9 mm to (104.3, 72.9)
- moved TP3 97.6 mm to (59.8, 66.4)
- moved C5 94.9 mm to (61.5, 82.1)
- moved R6 91.4 mm to (65.8, 75.2), turned to 180 degrees
- moved TP1 89.9 mm to (55.9, 73.0)
- moved R5 88.5 mm to (68.2, 75.2), turned to 180 degrees
- moved R2 88.5 mm to (61.3, 75.2)
- moved R16 88.1 mm to (70.8, 80.0), turned to 90 degrees
- moved TP5 87.9 mm to (70.9, 93.0)
- moved C3 87.6 mm to (71.2, 77.9)
- moved R15 87.5 mm to (70.3, 86.4)
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- renumbered SW4 to BOOT0, SW1 to NRST
Routing:
- net +3.3V: track 20.8 -> 73.7 mm, vias 2 -> 31
- net GND: track 8.31 -> 61.1 mm, vias 1 -> 53
- net /STM32H735/NRST: track 0.00 -> 51.3 mm, vias 0 -> 3
- net /STM32H735/USR_LED_1: track 0.00 -> 47.9 mm
- net /STM32H735/USR_LED_2: track 0.00 -> 46.3 mm
- net /STM32H735/USR_LED_3: track 0.00 -> 44.9 mm
- net /STM32H735/USR_LED_4: track 0.00 -> 42.6 mm
- net /STM32H735/TX2: track 0.00 -> 31.8 mm
- net /STM32H735/RX2: track 0.00 -> 29.8 mm
- net +5V: track 0.00 -> 23.3 mm, vias 0 -> 16
- net /STM32H735/USB_DM: track 0.00 -> 22.1 mm, vias 0 -> 1
- net /STM32H735/USB_DP: track 0.00 -> 22.0 mm, vias 0 -> 1
- net /GPIO14_TXD: track 0.00 -> 21.9 mm, vias 0 -> 1
- net /STM32H735/TX10: track 0.00 -> 21.5 mm, vias 0 -> 1
- net /GPIO15_RXD: track 0.00 -> 20.1 mm, vias 0 -> 1
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- added copper zone on B.Cu, net +3.3V
- added copper zone on B.Cu, net +3.3VA
- added copper zone on B.Cu, net +5V
- added copper zone on B.Cu, net Net-(U3-FB)
- added copper zone on B.Cu, net Net-(U3-SW)

Commit message: Mainboard Done !
Parts:
- removed J1: USB_C_Receptacle_USB2.0_16P, Connector_USB:USB_C_Receptacle_GCT_USB4110
- removed U2: USBLC6-2SC6, Package_TO_SOT_SMD:SOT-23-6
- LIDAR1, UART1, UART10, UART2, UART3, UART4, UART5, UART6, UART7, UART8: footprint Connector_JST:JST_XH_B4B-XH-A_1x04_P2.50mm_Vertical -> Connector_JST:JST_EH_B4B-EH-A_1x04_P2.50mm_Vertical
- SW2: renamed from USER BTN 1
- SW3: renamed from USER BTN2
- moved LIDAR1 7.68 mm to (100.8, 60.3), turned to 180 degrees
- moved D9 7.34 mm to (97.0, 56.5), turned to 90 degrees
- moved D8 2.55 mm to (82.5, 62.0)
- moved D6 1.60 mm to (66.7, 62.6)
- moved UART8 1.46 mm to (78.8, 59.6)
- moved UART6 1.10 mm to (63.5, 60.0)
- moved UART7 0.83 mm to (94.2, 100.8)
- moved UART10 0.74 mm to (61.2, 100.7)
- moved UART4 0.70 mm to (77.8, 100.7)
- moved UART3 0.39 mm to (108.7, 95.2)
- moved UART1 0.27 mm to (108.7, 67.8)
- moved UART5 0.27 mm to (108.7, 81.5)
- renumbered NRST to SW1, BOOT0 to SW4
Routing:
- net /STM32H735/USB_DM: track 22.1 -> 0.00 mm, vias 1 -> 0
- net /STM32H735/USB_DP: track 22.0 -> 0.00 mm, vias 1 -> 0
- net Net-(J1-D+-PadA6): track 11.9 -> 0.00 mm
- net Net-(J1-D--PadA7): track 11.9 -> 0.00 mm
- net GND: track 61.1 -> 49.3 mm, vias 53 -> 445
- net +3.3V: track 73.7 -> 82.3 mm
- net /STM32H735/TX_Lidar: track 10.2 -> 16.7 mm
- net /STM32H735/RX_Lidar: track 10.2 -> 12.5 mm
- net /STM32H735/RX5: track 14.4 -> 15.7 mm
- net /STM32H735/RX6: track 24.7 -> 23.6 mm
- net /STM32H735/TX6: track 27.5 -> 26.4 mm
- net /STM32H735/USR_LED_1: track 47.9 -> 47.1 mm
- net /STM32H735/USR_LED_2: track 46.3 -> 45.6 mm
- net /STM32H735/TX8: track 22.5 -> 21.9 mm
- net /STM32H735/RX7: track 33.8 -> 33.2 mm

Commit message: Updating t
Parts:
- C12, C13, C14, C15, C16, C17, C18, C19, C20, C21, C22, C23, C24, C25, C26, C27, C28, C3, C40, C42, C43, C44, C45, C46, C47, C5: footprint Capacitor_SMD:C_0402_1005Metric_Pad0.74x0.62mm_HandSolder -> Capacitor_SMD:C_0402_1005Metric
- C29: footprint Capacitor_SMD:C_0603_1608Metric_Pad1.08x0.95mm_HandSolder -> Capacitor_SMD:C_0603_1608Metric
- C34, C4, C6, C8: footprint Capacitor_SMD:C_0603_1608Metric_Pad1.08x0.95mm_HandSolder -> Capacitor_SMD:C_0402_1005Metric
- C37: footprint Capacitor_SMD:C_0805_2012Metric_Pad1.18x1.45mm_HandSolder -> Capacitor_SMD:C_0805_2012Metric
- C38: footprint Capacitor_SMD:C_0805_2012Metric_Pad1.18x1.45mm_HandSolder -> Capacitor_SMD:C_0402_1005Metric
- F1: footprint Fuse:Fuse_1206_3216Metric_Pad1.42x1.75mm_HandSolder -> Fuse:Fuse_1206_3216Metric
- R1: footprint Resistor_SMD:R_0805_2012Metric_Pad1.20x1.40mm_HandSolder -> Resistor_SMD:R_0402_1005Metric
- R2, R3, R5, R6: footprint Resistor_SMD:R_0402_1005Metric_Pad0.72x0.64mm_HandSolder -> Resistor_SMD:R_0402_1005Metric
- moved LIDAR1 7.26 mm to (93.5, 60.0), turned to 0 degrees
- moved D9 6.51 mm to (97.5, 63.0), turned to -90 degrees
- moved R1 1.18 mm to (53.2, 80.0)
- moved UART8 0.40 mm to (78.8, 60.0)
Routing:
- net /STM32H735/TX_Lidar: track 16.7 -> 11.5 mm
- net /STM32H735/RX8: track 18.5 -> 15.8 mm
- net /STM32H735/RX_Lidar: track 12.5 -> 11.1 mm
- net GND: vias 445 -> 444
Other:
- board text added: "24V"
- board text added: "GND"
- board text added: "RX"
- board text added: "TX"

Commit message: Edits of the PCB done
Routing:
- net GND: vias 444 -> 443
