File: Hardware/Hardware_électronique/MainBoard/PCB_test/MainBoard_test1/test1.kicad_sch (KiCad schematic)
At the start: 2 parts

Commit message: commitment
Parts:
- added ARU2: 180G-2, MainBoard:180G-2, symbol schematic1-eagle-import:180G-2
- added BT1: Battery, symbol Device:Battery
- added C1: C_Polarized_Small, schematic1:E5-6, symbol Device:C_Polarized_Small
- added D10: 1.5SMBJ36CA, Diode_SMD:D_SMB, symbol Device:D_TVS
- added D11: 4V7, Diode_SMD:D_0603_1608Metric, symbol Device:D_Zener_Small
- added D14, D15, D16, D17: LED, LED_SMD:LED_0603_1608Metric, symbol Device:LED
- added F1: 15A, Fuse:Fuse_1206_3216Metric_Pad1.42x1.75mm_HandSolder, symbol Device:Fuse_Small
- added J1: Conn_RasPi, Connector_PinSocket_2.54mm:PinSocket_2x20_P2.54mm_Vertical, symbol Connector_Generic:Conn_02x20_Odd_Even
- added Q1: PMOS, schematic1:MOS_WDFN8, symbol Device:Q_PMOS_GDS
- added R1: 10k, Resistor_SMD:R_0805_2012Metric_Pad1.20x1.40mm_HandSolder, symbol Device:R_Small
- added R10, R11: 1k, Resistor_SMD:R_0402_1005Metric, symbol Device:R_Small
- added R8: 6k2, Resistor_SMD:R_0402_1005Metric, symbol Device:R_Small
- added R9: 1k8, Resistor_SMD:R_0402_1005Metric, symbol Device:R_Small
- added TP1: TestPoint, symbol Connector:TestPoint
Connections:
- net VBUS: now also C1.1, D11.1 (K), Q1.3 (S), R8.1, TP1.1
- new net: D17.2 (A), R11.2
- new net: ARU2.2, D10.2 (A2), Q1.2 (D)
- new net: D15.2 (A), R9.2
- new net: D16.2 (A), R10.2
- new net: D11.2 (A), Q1.1 (G), R1.1
- new net: BT1.1 (+), F1.1
- new net: D14.2 (A), R8.2
- new net +3.3V: R11.1
- new net +BATT: ARU2.1, F1.2
- new net 5.1V: R10.1
- new net 5V: J1.2 (Pin_2), J1.4 (Pin_4)
- new net 7.5V: R9.1
- new net GND: BT1.2 (-), C1.2, D10.1 (A1), D14.1 (K), D15.1 (K), D16.1 (K), D17.1 (K), J1.14 (Pin_14), J1.6 (Pin_6), J1.9 (Pin_9), R1.2
- new net GPIO0_ID_SD: J1.27 (Pin_27)
- new net GPIO10_MOSI: J1.19 (Pin_19)
- new net GPIO11_SCLK: J1.23 (Pin_23)
- new net GPIO12_PWM0: J1.32 (Pin_32)
- new net GPIO13_PWM1: J1.33 (Pin_33)
- new net GPIO14_TXD: J1.8 (Pin_8)
- new net GPIO15_RXD: J1.10 (Pin_10)
- new net GPIO16: J1.36 (Pin_36)
- new net GPIO17: J1.11 (Pin_11)
- new net GPIO18_PCMCLK: J1.12 (Pin_12)
- new net GPIO19_PCMFS: J1.35 (Pin_35)
- new net GPIO1_ID_SD: J1.28 (Pin_28)
- new net GPIO20_PCMDIN: J1.38 (Pin_38)
- new net GPIO21_PCMDOUT: J1.40 (Pin_40)
- new net GPIO22: J1.15 (Pin_15)
- new net GPIO23: J1.16 (Pin_16)
- new net GPIO24: J1.18 (Pin_18)
- new net GPIO25: J1.22 (Pin_22)
- new net GPIO26: J1.37 (Pin_37)
- new net GPIO27: J1.13 (Pin_13)
- new net GPIO2_SDA: J1.3 (Pin_3)
- new net GPIO3_SCL: J1.5 (Pin_5)
- new net GPIO4_GPCLK0: J1.7 (Pin_7)
- new net GPIO5: J1.29 (Pin_29)
- new net GPIO6: J1.31 (Pin_31)
- new net GPIO7_CE1: J1.26 (Pin_26)
- new net GPIO8_CE0: J1.24 (Pin_24)
- new net GPIO9_MISO: J1.21 (Pin_21)
- no-connect marks 0 -> 7
Other:
- removed sheet Alimentation
- removed sheet Conn_ext
- removed sheet RaspberryPi4
- sheet STM32H735 ports: added RXtoRPI, TXtoRPI; removed none
- note added: "CONNECTEUR BAT"
- note added: "LED"

Commit message: hey
Parts:
- BT1: footprint (none) -> Connector_AMASS:AMASS_XT60PW-F_1x02_P7.20mm_Horizontal
- TP1, TP3, TP4: footprint (none) -> TestPoint:TestPoint_Pad_D2.0mm
Changed lines of the file:
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@@
 	(wire
 		(pts
+			(xy 67.31 33.02) (xy 80.01 33.02)
+		)
+		(stroke
+			(width 0)
+			(type default)
+		)
+	)
+	(wire
+		(pts
 			(xy 69.215 139.7) (xy 69.215 140.335)
 		)
@@
 	(wire
 		(pts
+			(xy 67.31 30.48) (xy 80.01 30.48)
+		)
+		(stroke
+			(width 0)
+			(type default)
+		)
+	)
+	(wire
+		(pts
 			(xy 74.93 138.43) (xy 74.93 140.335)
 		)
@@
 		)
 	)
-	(label "GPIO15_TXD"
+	(label "GPIO15_RXD"
+		(at 80.01 33.02 180)
+		(fields_autoplaced yes)
+		(effects
+			(font
+				(size 1.27 1.27)
+			)
+			(justify right bottom)
+		)
+	)
+	(label "GPIO15_RXD"
 		(at 100.33 46.99 0)
 		(fields_autoplaced yes)
@@
 		)
 	)
-	(label "GPIO15_RXD"
+	(label "GPIO14_TXD"
 		(at 100.33 44.45 0)
 		(fields_autoplaced yes)
@@
 		)
 	)
+	(label "GPIO14_TXD"
+		(at 80.01 30.48 180)
+		(fields_autoplaced yes)
+		(effects
+			(font
+				(size 1.27 1.27)
+			)
+			(justify right bottom)
+		)
+	)
 	(global_label "GPIO16"
 		(shape input)
@@
 		)
 	)
-	(global_label "GPIO14_TXD"
-		(shape input)
-		(at 67.31 30.48 0)
-		(fields_autoplaced yes)
-		(effects
-			(font
-				(size 1.27 1.27)
-			)
-			(justify left)
-		)
-		(property "Intersheetrefs" "${INTERSHEET_REFS}"
-			(at 81.6042 30.48 0)
-			(effects
-				(font
-					(size 1.27 1.27)
-				)
-				(justify left)
-				(hide yes)
-			)
-		)
-	)
 	(global_label "GPIO5"
 		(shape input)
@@
 		)
 	)
-	(global_label "GPIO15_RXD"
-		(shape input)
-		(at 67.31 33.02 0)
-		(fields_autoplaced yes)
-		(effects
-			(font
-				(size 1.27 1.27)
-			)
-			(justify left)
-		)
-		(property "Intersheetrefs" "${INTERSHEET_REFS}"
-			(at 81.9066 33.02 0)
-			(effects
-				(font
-					(size 1.27 1.27)
-				)
-				(justify left)
-				(hide yes)
-			)
-		)
-	)
 	(global_label "GPIO17"
 		(shape input)
@@
 			)
 		)
-		(property "Footprint" ""
+		(property "Footprint" "TestPoint:TestPoint_Pad_D2.0mm"
 			(at 48.26 88.9 0)
 			(effects
@@
 			)
 		)
-		(property "Footprint" ""
+		(property "Footprint" "Connector_AMASS:AMASS_XT60PW-F_1x02_P7.20mm_Horizontal"
 			(at 34.29 136.906 90)
 			(effects
@@
 			)
 		)
-		(property "Footprint" ""
+		(property "Footprint" "TestPoint:TestPoint_Pad_D2.0mm"
 			(at 46.99 102.87 0)
 			(effects
@@
 			)
 		)
-		(property "Footprint" ""
+		(property "Footprint" "TestPoint:TestPoint_Pad_D2.0mm"
 			(at 95.885 132.08 0)
 			(effects

Commit message: approaching end of schematics
Parts:
- removed D15: LED, LED_SMD:LED_0603_1608Metric, symbol Device:LED
- removed R9: 1k8, Resistor_SMD:R_0402_1005Metric, symbol Device:R_Small
- removed TP4: TestPoint, TestPoint:TestPoint_Pad_D2.0mm, symbol Connector:TestPoint
Connections:
- net 5.1V is gone; now on net +5V: R10.1
- net 5V is gone; now on net +5V: J1.2 (Pin_2), J1.4 (Pin_4)
- net +BATT: now also ARU2.2, D10.2 (A2), Q1.2 (D); no longer ARU2.1, F1.2
- net GPIO0_ID_SD: no longer names the net of J1.27 (Pin_27)
- net GPIO10_MOSI: no longer names the net of J1.19 (Pin_19)
- net GPIO11_SCLK: no longer names the net of J1.23 (Pin_23)
- net GPIO12_PWM0: no longer names the net of J1.32 (Pin_32)
- net GPIO13_PWM1: no longer names the net of J1.33 (Pin_33)
- net GPIO16: no longer names the net of J1.36 (Pin_36)
- net GPIO17: no longer names the net of J1.11 (Pin_11)
- net GPIO18_PCMCLK: no longer names the net of J1.12 (Pin_12)
- net GPIO19_PCMFS: no longer names the net of J1.35 (Pin_35)
- net GPIO1_ID_SD: no longer names the net of J1.28 (Pin_28)
- net GPIO20_PCMDIN: no longer names the net of J1.38 (Pin_38)
- net GPIO21_PCMDOUT: no longer names the net of J1.40 (Pin_40)
- net GPIO22: no longer names the net of J1.15 (Pin_15)
- net GPIO23: no longer names the net of J1.16 (Pin_16)
- net GPIO24: no longer names the net of J1.18 (Pin_18)
- net GPIO25: no longer names the net of J1.22 (Pin_22)
- net GPIO26: no longer names the net of J1.37 (Pin_37)
- net GPIO27: no longer names the net of J1.13 (Pin_13)
- net GPIO2_SDA: no longer names the net of J1.3 (Pin_3)
- net GPIO3_SCL: no longer names the net of J1.5 (Pin_5)
- net GPIO4_GPCLK0: no longer names the net of J1.7 (Pin_7)
- net GPIO5: no longer names the net of J1.29 (Pin_29)
- net GPIO6: no longer names the net of J1.31 (Pin_31)
- net GPIO7_CE1: no longer names the net of J1.26 (Pin_26)
- net GPIO8_CE0: no longer names the net of J1.24 (Pin_24)
- net GPIO9_MISO: no longer names the net of J1.21 (Pin_21)
- new net: ARU2.1, F1.2
- no-connect marks 7 -> 33
Other:
- removed sheet Buck7.5
- note added: "Conn Raspberry Pi 4"
- moved on the sheet: ARU2, BT1, C1, D10, D11, D14, D16, D17, F1, Q1, R1, R10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

Commit message: quite finished schematics
Parts:
- removed ARU2: 180G-2, MainBoard:180G-2, symbol schematic1-eagle-import:180G-2
- added ARU1: 180G-2, MainBoard:180G-2, symbol schematic1-eagle-import:180G-2
- F1: footprint Fuse:Fuse_1206_3216Metric_Pad1.42x1.75mm_HandSolder -> (none); Mouser Part Number 693-3413.0330.22 -> (none)
Connections:
- net +BATT: now also ARU1.2
- net at F1.2: now also ARU1.1
Other:
- moved on the sheet: D14, D16, D17, R10, R11, R8
