File: 2A/Hardware/Hardware_électronique/Auxiliairy_board/PCB_Moteur/Inverter_KiCAD/Inverter_KiCAD.kicad_pcb (KiCad board)
At the start: 4 copper layers, 70 x 70 mm, 109 parts, among them J1 Conn_02x02_Top_Bottom, J2 173010542, J3 Conn_02x05_Odd_Even, J4 Conn_01x02, J5 Conn_01x02, J6 Conn_ST_STDC14, J7 Conn_01x04_Pin, Q5 SQ2310ES, SW1 SW_Push, SW2 SW_Push, SW7 SW_Push, SW8 SW_Push, U1 MIC4606, U1201 TCN75A, U2 GO 10-SME/SP3, U3 GO 10-SME/SP3, U4 AZ1117-3.3, U5 MAX3097ECSE+, U6 STM32G474RETx, U7 CSD86350Q5D, U8 CSD86350Q5D, Y1 16M

Commit message: Add files via upload
Parts:
- removed C33: 10u, Capacitor_SMD:C_0603_1608Metric_Pad1.08x0.95mm_HandSolder
- removed C34: 4.7nF, Capacitor_SMD:C_0402_1005Metric_Pad0.74x0.62mm_HandSolder
- removed C35: 22nF, Capacitor_SMD:C_0402_1005Metric
- removed C36: 47u, Capacitor_SMD:C_0805_2012Metric
- removed R26: 287k, Resistor_SMD:R_0402_1005Metric
- removed R27: 1.91k, Resistor_SMD:R_0402_1005Metric
- removed R28: 34k, Resistor_SMD:R_0402_1005Metric
- removed TP 5V: TestPoint, TestPoint:TestPoint_Pad_D2.0mm
- removed TP 7.5V: TestPoint, TestPoint:TestPoint_Pad_D2.0mm
- removed WPMDH1302401: ~, Package_TO_SOT_SMD:TO-263-7_TabPin8
- added C11: 10u, Capacitor_SMD:C_2220_5750Metric, B.Cu at (159.2, 123.4)
- added C12: 10u, Capacitor_SMD:C_2220_5750Metric, B.Cu at (153.2, 123.5)
- added C37: 2.2n, Capacitor_SMD:C_0402_1005Metric, B.Cu at (152.0, 111.4)
- added C40: 100n, Capacitor_SMD:C_0402_1005Metric, B.Cu at (159.5, 116.6)
- added C41: 22u, Capacitor_SMD:C_0805_2012Metric, B.Cu at (161.9, 107.8)
- added C42: 22u, Capacitor_SMD:C_0805_2012Metric, B.Cu at (161.9, 105.8)
- added C43: 22u, Capacitor_SMD:C_0805_2012Metric, B.Cu at (165.7, 107.8)
- added G***1: LOGO, PCBAres:logo, F.Cu at (190.8, 141.4)
- added G***1: LOGO, PCBAres:logo, B.Cu at (190.7, 141.5)
- added L2: 4.7u, MainBoard:PA5432.472NLT, B.Cu at (162.5, 112.6)
- added R2: 200k, Resistor_SMD:R_0402_1005Metric, B.Cu at (152.0, 115.4)
- added R29: 19.6k, Resistor_SMD:R_0402_1005Metric, B.Cu at (154.3, 110.8)
- added R30: 12.1k, Resistor_SMD:R_0402_1005Metric, B.Cu at (156.5, 110.3)
- added R31: 1.5k, Resistor_SMD:R_0402_1005Metric, B.Cu at (156.0, 108.8)
- added TP2: 7.5V, TestPoint:TestPoint_Pad_D2.0mm, F.Cu at (164.5, 119.7)
- added TP3: 5V, TestPoint:TestPoint_Pad_D2.0mm, F.Cu at (189.1, 127.5)
- added U9: AP64500Q, Package_SO:SOIC-8-1EP_3.9x4.9mm_P1.27mm_EP2.95x4.9mm_Mask2.71x3.4mm, B.Cu at (155.4, 115.2)
- C1, C4: footprint Capacitor_SMD:C_0603_1608Metric_Pad1.08x0.95mm_HandSolder -> Capacitor_SMD:C_2220_5750Metric
- C10, C8, C9: footprint Capacitor_SMD:CP_Elec_10x10.5 -> Capacitor_SMD:C_1210_3225Metric
- C2, C3: footprint Capacitor_SMD:C_0603_1608Metric_Pad1.08x0.95mm_HandSolder -> Capacitor_SMD:C_0805_2012Metric
- J1: value Conn_02x02_Top_Bottom -> Conn_Motor; footprint Connector_Molex:Molex_Micro-Fit_3.0_43045-0400_2x02_P3.00mm_Horizontal -> Connector_AMASS:AMASS_XT30PW-M_1x02_P2.50mm_Horizontal
- J3: footprint Connector_PinHeader_2.54mm:PinHeader_2x05_P2.54mm_Vertical -> Connector_PinHeader_1.27mm:PinHeader_2x05_P1.27mm_Vertical_SMD
- TP4: value TestPoint -> 3.3V
- moved C8 18.1 mm to (151.7, 125.6), turned to -90 degrees
- moved C10 16.3 mm to (153.8, 120.6), turned to 90 degrees
- moved C19 11.2 mm to (160.1, 109.0), turned to -90 degrees
- moved C9 9.23 mm to (150.4, 120.6), turned to 90 degrees
- moved U5 9.03 mm to (165.9, 111.3)
- moved J2 8.53 mm to (164.1, 123.4), turned to 0 degrees
- moved TP1 6.93 mm to (155.0, 124.8)
- moved J1 6.33 mm to (170.8, 135.2)
- moved C4 3.60 mm to (171.2, 119.5), turned to 90 degrees
- moved J3 3.01 mm to (159.1, 141.8), turned to 180 degrees
- moved C1 2.55 mm to (185.0, 119.7), turned to 90 degrees
- moved R7 2.32 mm to (180.4, 116.9), turned to 180 degrees
- moved D5 1.30 mm to (180.3, 115.5)
- moved R8 1.10 mm to (183.1, 113.9)
- moved D1 1.10 mm to (180.3, 110.5)
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Connections:
- J1 pad 1: /ARM_OUT_A -> /ARM_B
- J1 pad 2: GND -> /ARM_OUT_A
Routing:
- net +7.5V: track 51.8 -> 23.0 mm, vias 2 -> 0
- net VBUS: track 27.9 -> 2.02 mm, vias 50 -> 21
- net //Z: track 41.4 -> 30.2 mm, vias 1 -> 0
- net GND: track 30.1 -> 19.1 mm, vias 68 -> 158
- net Net-(U9-FB): track 0.00 -> 10.9 mm
- net Net-(Converter_DCDC_WPMDH1302401-FB): track 7.38 -> 0.00 mm
- net /Z: track 38.0 -> 31.1 mm, vias 1 -> 0
- net //B: track 40.0 -> 34.8 mm, vias 1 -> 2
- net Net-(Converter_DCDC_WPMDH1302401-SS): track 3.75 -> 0.00 mm
- net Net-(Converter_DCDC_WPMDH1302401-RON): track 3.52 -> 0.00 mm
- net /ENC_C: track 11.6 -> 14.7 mm
- net /B: track 36.3 -> 33.3 mm, vias 1 -> 0
- net //A: track 38.6 -> 35.6 mm, vias 1 -> 2
- net /Imes_vbus: track 55.2 -> 57.8 mm, vias 0 -> 2
- net Net-(U9-RT/CLK): track 0.00 -> 2.52 mm
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- added copper zone on B.Cu, net Net-(U9-SW)
- added copper zone on B.Cu, net VBUS
- removed copper zone on B.Cu, net (none)
- removed copper zone on F.Cu, net (none)
Other:
- board text added: "PCB_Moteur_v2 By Kenny Saint Fleur"

Commit message: pcb edits
Parts:
- removed C11, C12: 10u, Capacitor_SMD:C_2220_5750Metric
- removed C37: 2.2n, Capacitor_SMD:C_0402_1005Metric
- removed C40: 100n, Capacitor_SMD:C_0402_1005Metric
- removed C41, C42, C43: 22u, Capacitor_SMD:C_0805_2012Metric
- removed D4, D6, D7: Red LED, LED_SMD:LED_0603_1608Metric
- removed J2: 173010542, Connector_PinHeader_2.54mm:PinHeader_1x03_P2.54mm_Vertical
- removed L2: 4.7u, MainBoard:PA5432.472NLT
- removed R2: 200k, Resistor_SMD:R_0402_1005Metric
- removed R29: 19.6k, Resistor_SMD:R_0402_1005Metric
- removed R30: 12.1k, Resistor_SMD:R_0402_1005Metric
- removed R31: 1.5k, Resistor_SMD:R_0402_1005Metric
- removed R4, R8: 390, Resistor_SMD:R_0402_1005Metric
- removed R9: 680, Resistor_SMD:R_0402_1005Metric
- removed TP1: TestPoint, TestPoint:TestPoint_Pad_D2.0mm
- removed TP2: 7.5V, TestPoint:TestPoint_Pad_D2.0mm
- removed TP3: 5V, TestPoint:TestPoint_Pad_D2.0mm
- removed TP4: 3.3V, TestPoint:TestPoint_Pad_D2.0mm
- removed U4: AZ1117-3.3, Package_TO_SOT_SMD:SOT-223-3_TabPin2
- removed U9: AP64500Q, Package_SO:SOIC-8-1EP_3.9x4.9mm_P1.27mm_EP2.95x4.9mm_Mask2.71x3.4mm
- added BU33SD5WG-TR1: LM1117DT-3.3, Package_TO_SOT_SMD:SOT-23-5, F.Cu at (195.2, 125.1)
- added C102: 1u, Capacitor_SMD:C_0603_1608Metric, B.Cu at (158.5, 118.0)
- added C103: 47u, Capacitor_SMD:C_0805_2012Metric, B.Cu at (165.7, 116.0)
- added C404: 2u2, Capacitor_SMD:C_0603_1608Metric, B.Cu at (176.3, 119.4)
- added R101: 1k8, Resistor_SMD:R_0402_1005Metric, B.Cu at (155.2, 117.4)
- added R102: 20k, Resistor_SMD:R_0402_1005Metric, B.Cu at (157.5, 116.0)
- added R103: 2k, Resistor_SMD:R_0402_1005Metric, B.Cu at (156.3, 117.4)
- added R403: 0R3, Resistor_SMD:R_1210_3225Metric, B.Cu at (184.1, 126.8)
- added R404: 0R3, Resistor_SMD:R_1210_3225Metric, B.Cu at (173.2, 120.4)
- added TP3V3: TestPoint_Small, TestPoint:TestPoint_Pad_D1.0mm, B.Cu at (194.2, 121.0)
- added TP9V1: 3.3V, TestPoint:TestPoint_Pad_D1.0mm, B.Cu at (164.0, 118.2)
- added TPBOOT0-1: TestPoint_Small, TestPoint:TestPoint_Pad_D1.0mm, B.Cu at (182.2, 92.1)
- added U101: WPME-VDLM, CustomLibrary:WPME-VDLM, B.Cu at (159.8, 122.3)
- C10, C8: footprint Capacitor_SMD:C_1210_3225Metric -> Capacitor_SMD:C_Elec_10x10.2
- C17: value 10u -> 1u
- C18: value 22u -> 1u
- C9: value 220u -> 10u; footprint Capacitor_SMD:C_1210_3225Metric -> Capacitor_SMD:C_2220_5750Metric; moved to B.Cu
- J1: footprint Connector_AMASS:AMASS_XT30PW-M_1x02_P2.50mm_Horizontal -> Connector_AMASS:AMASS_XT30UPB-F_1x02_P5.0mm_Vertical
- U1: footprint Package_SO:TSSOP-16-1EP_4.4x5mm_P0.65mm_EP3x3mm -> Package_SO:TSSOP-16_4.4x5mm_P0.65mm
- moved C18 8.44 mm to (191.5, 123.9), turned to 180 degrees
- moved R10 7.41 mm to (198.4, 124.4), turned to -90 degrees
- moved BT1 7.15 mm to (144.9, 136.3), turned to 90 degrees
- moved C8 5.67 mm to (156.0, 129.3)
- moved C10 4.65 mm to (152.3, 116.2)
- moved C17 4.02 mm to (191.5, 126.2), turned to 180 degrees
- moved R7 3.21 mm to (180.6, 113.7)
- moved D5 3.20 mm to (180.2, 112.3)
- moved C9 3.07 mm to (151.4, 117.7)
- moved C23 1.87 mm to (194.3, 96.9), turned to -90 degrees
- moved D8 1.70 mm to (198.4, 121.8), turned to 90 degrees
- moved C30 1.00 mm to (192.7, 96.5), turned to -90 degrees
- moved C5 0.98 mm to (188.7, 131.1), turned to 0 degrees
- moved R1 0.80 mm to (180.6, 109.2)
- moved C3 0.36 mm to (179.8, 111.7)
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Connections:
- net /MCU_STM32G475/NRST renamed /MCU_STM32G474/NRST
- net /MCU_STM32G475/SWCLK renamed /MCU_STM32G474/SWCLK
- net /MCU_STM32G475/SWDIO renamed /MCU_STM32G474/SWDIO
- net /MCU_STM32G475/SWO renamed /MCU_STM32G474/SWO
- net /MCU_STM32G475/USART1_RX renamed /MCU_STM32G474/USART1_RX
- net /MCU_STM32G475/USART1_TX renamed /MCU_STM32G474/USART1_TX
- net /MCU_STM32G475/USR_BTN_1 renamed /MCU_STM32G474/USR_BTN_1
- net /MCU_STM32G475/USR_LED_1 renamed /MCU_STM32G474/USR_LED_1
- net /MCU_STM32G475/USR_LED_2 renamed /MCU_STM32G474/USR_LED_2
- net /MCU_STM32G475/USR_LED_3 renamed /MCU_STM32G474/USR_LED_3
- net /MCU_STM32G475/USR_LED_4 renamed /MCU_STM32G474/USR_LED_4
- net /MCU_STM32G475/VCP_RX renamed /MCU_STM32G474/VCP_RX
- net /MCU_STM32G475/VCP_TX renamed /MCU_STM32G474/VCP_TX
- BT1 pad 1: Net-(BT1-+) -> GND
- BT1 pad 2: GND -> Net-(BT1-+)
- C17 pad 1: +5V -> +9V
- C20 pad 2: /MCU_STM32G475/USR_BTN_2 -> /MCU_STM32G474/USR_BTN_2
- C39 pad 2: /MCU_STM32G475/USR_BTN_3 -> /MCU_STM32G474/USR_BTN_3
- J4 pad 1: +5V -> +9V
- J5 pad 1: +5V -> +9V
- R13 pad 2: /MCU_STM32G475/USR_BTN_2 -> /MCU_STM32G474/USR_BTN_2
- R24 pad 2: /MCU_STM32G475/USR_BTN_3 -> /MCU_STM32G474/USR_BTN_3
- U1 pad 10: /ARM_IN_A -> Net-(U1-AHS)
- U1 pad 12: +7.5V -> +9V
- U1 pad 15: /ARM_B -> Net-(U1-BHS)
- U1 pad 4: /In_B_L -> unconnected-(U1-BLI-Pad4)
- U1 pad 5: /In_A_L -> unconnected-(U1-ALI-Pad5)
- U6 pad 10: /ENC_C -> unconnected-(U6-PC2-Pad10)
- U6 pad 11: unconnected-(U6-PC3-Pad11) -> /Pwr_EN
- U6 pad 12: unconnected-(U6-PA0-Pad12) -> /ENC_A
- U6 pad 13: /Imes_mot -> /ENC_B
- U6 pad 14: /In_A_H -> unconnected-(U6-PA2-Pad14)
- U6 pad 17: /In_A_L -> unconnected-(U6-PA3-Pad17)
- U6 pad 18: /MCU_STM32G475/USR_BTN_2 -> unconnected-(U6-PA4-Pad18)
- U6 pad 19: unconnected-(U6-PA5-Pad19) -> /ENC_C
- U6 pad 2: /Pwr_EN -> unconnected-(U6-PC13-Pad2)
- U6 pad 21: unconnected-(U6-PA7-Pad21) -> /In_B_H
- U6 pad 25: unconnected-(U6-PB1-Pad25) -> /PWM_FAN
- U6 pad 26: unconnected-(U6-PB2-Pad26) -> /Imes_mot
- U6 pad 36: /Imes_vbus -> unconnected-(U6-PB14-Pad36)
- U6 pad 38: /In_B_H -> unconnected-(U6-PC6-Pad38)
- U6 pad 39: /In_B_L -> unconnected-(U6-PC7-Pad39)
- U6 pad 57: /PWM_FAN -> /MCU_STM32G474/USR_BTN_2
- U6 pad 58: unconnected-(U6-PB5-Pad58) -> /MCU_STM32G474/USR_BTN_3
- U6 pad 59: /MCU_STM32G475/USR_BTN_3 -> unconnected-(U6-PB6-Pad59)
- U6 pad 8: /ENC_A -> /In_A_H
- U6 pad 9: /ENC_B -> /Imes_vbus
Routing:
- net GND: track 19.1 -> 63.3 mm, vias 158 -> 165
- net +9V: track 0.00 -> 31.4 mm, vias 0 -> 7
- net /MCU_STM32G475/USR_BTN_2: track 29.9 -> 0.00 mm, vias 2 -> 0
- net /In_B_L: track 29.3 -> 0.00 mm, vias 2 -> 0
- net +7.5V: track 23.0 -> 0.00 mm
- net /MCU_STM32G475/USR_BTN_3: track 18.4 -> 0.00 mm
- net /MCU_STM32G474/USR_BTN_3: track 0.00 -> 17.2 mm
- net /In_B_H: track 33.3 -> 17.6 mm, vias 2 -> 1
- net /In_A_L: track 15.5 -> 0.00 mm, vias 1 -> 0
- net Net-(U1-AHS): track 0.00 -> 13.2 mm
- net /Imes_vbus: track 57.8 -> 44.9 mm, vias 2 -> 0
- net /MCU_STM32G474/USR_BTN_2: track 0.00 -> 11.0 mm
- net Net-(U9-FB): track 10.9 -> 0.00 mm
- net /MCU_STM32G474/SWO: track 30.6 -> 21.2 mm
- net /MCU_STM32G474/SWCLK: track 26.4 -> 18.9 mm
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- added copper zone on B.Cu, net +9V
- added copper zone on In2.Cu, net +9V
- removed copper zone on In2.Cu, net +5V
- removed copper zone on B.Cu, net +7.5V
- removed copper zone on B.Cu, net Net-(U9-SW)
Other:
- board text added: "PCB_Moteur_v3 By Kenny Saint Fleur"
- board text removed: "PCB_Moteur_v2 By Kenny Saint Fleur"
