File: 2A/Hardware/Hardware_électronique/Auxiliairy_board/PCB_Moteur/Inverter_KiCAD/Inverter_KiCAD.kicad_sch (KiCad schematic)
At the start: 65 parts, among them J1 Conn_02x02_Top_Bottom, J2 173010542, J3 Conn_02x05_Odd_Even, J4 Conn_01x02, J5 Conn_01x02, Q5 SQ2310ES, U1 MIC4606, U2 GO 10-SME/SP3, U3 GO 10-SME/SP3, U4 AZ1117-3.3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

Commit message: Add files via upload
Parts:
- removed C33: 10u, Capacitor_SMD:C_0603_1608Metric_Pad1.08x0.95mm_HandSolder, symbol Device:C
- removed C34: 4.7nF, Capacitor_SMD:C_0402_1005Metric_Pad0.74x0.62mm_HandSolder, symbol Device:C
- removed C35: 22nF, Capacitor_SMD:C_0402_1005Metric, symbol Device:C
- removed C36: 47u, Capacitor_SMD:C_0805_2012Metric, symbol Device:C
- removed Converter_DCDC_WPMDH1302401: ~, Package_TO_SOT_SMD:TO-263-7_TabPin8, symbol Custom:Converter_DCDC
- removed J1: Conn_02x02_Top_Bottom, Connector_Molex:Molex_Micro-Fit_3.0_43045-0400_2x02_P3.00mm_Horizontal, symbol Connector_Generic:Conn_02x02_Top_Bottom
- removed R26: 100k, Resistor_SMD:R_0402_1005Metric, symbol Device:R
- removed R27: 4.3k, Resistor_SMD:R_0402_1005Metric, symbol Device:R
- removed R28: 36k, Resistor_SMD:R_0402_1005Metric, symbol Device:R
- removed TP1: TestPoint, TestPoint:TestPoint_Pad_D2.0mm, symbol Connector:TestPoint
- added C11, C12: 10u, Capacitor_SMD:C_2220_5750Metric, symbol Device:C_Small
- added C37: 2.2n, Capacitor_SMD:C_0402_1005Metric, symbol Device:C_Small
- added C40: 100n, Capacitor_SMD:C_0402_1005Metric, symbol Device:C_Small
- added C41, C42, C43: 22u, Capacitor_SMD:C_0805_2012Metric, symbol Device:C_Small
- added J1: Conn_Motor, Connector_AMASS:AMASS_XT30PW-M_1x02_P2.50mm_Horizontal, symbol Connector_Generic:Conn_01x02
- added L2: 4.7u, MainBoard:PA5432.472NLT, symbol Device:L_Small
- added R2: 200k, Resistor_SMD:R_0402_1005Metric, symbol Device:R_Small
- added R29: 19.6k, Resistor_SMD:R_0402_1005Metric, symbol Device:R_Small
- added R30: 12.1k, Resistor_SMD:R_0402_1005Metric, symbol Device:R_Small
- added R31: 1.5k, Resistor_SMD:R_0402_1005Metric, symbol Device:R_Small
- added U9: AP64500Q, Package_SO:SOIC-8-1EP_3.9x4.9mm_P1.27mm_EP2.95x4.9mm_Mask2.71x3.4mm, symbol Custom:AP64500Q
- C1, C4: footprint Capacitor_SMD:C_0603_1608Metric_Pad1.08x0.95mm_HandSolder -> Capacitor_SMD:C_2220_5750Metric
- C10, C8, C9: footprint Capacitor_SMD:CP_Elec_10x10.5 -> Capacitor_SMD:C_1210_3225Metric; MFR 861 011 086 027 -> 885 012 209 043
- C2, C3: footprint Capacitor_SMD:C_0603_1608Metric_Pad1.08x0.95mm_HandSolder -> Capacitor_SMD:C_0805_2012Metric
- J3: footprint Connector_PinHeader_2.54mm:PinHeader_2x05_P2.54mm_Vertical -> Connector_PinHeader_1.27mm:PinHeader_2x05_P1.27mm_Vertical_SMD
- TP2: value TestPoint -> 7.5V
- TP3: value TestPoint -> 5V
- TP4: value TestPoint -> 3.3V
Connections:
- net +7.5V: now also C41.1, C42.1, C43.1, L2.2
- net ARM_B: now also J1.1 (Pin_1)
- net ARM_OUT_A: now also J1.2 (Pin_2)
- net GND: now also C11.1, C12.2, C37.2, C41.2, C42.2, C43.2, R2.2, R31.2, U9.7 (GND), U9.9 (EPad)
- net VBUS: now also C11.2, C12.1, U9.2 (VIN), U9.3 (EN)
- new net: C40.2, L2.1, R30.1, U9.8 (SW)
- new net: C37.1, R29.2
- new net: C40.1, U9.1 (BST)
- new net: R29.1, U9.6 (COMP)
- new net: R30.2, R31.1, U9.5 (FB)
- new net: R2.1, U9.4 (RT/CLK)
- no-connect marks 10 -> 9
Other:
- note added: "Buck 25.2V -> 7.5V"
- note added: "Wurth Capacitor : 885 012 209 043 220uF/50V"
- note removed: "ADD LDO for MIC4606"
- note removed: "ADD UREF"
- note removed: "SOULEVER PATE 3 AVANT DE SOUDER"
- note removed: "Wurth Capacitor : 865060657012 220uF/50V"
- moved on the sheet: C13, C14, C15, C17, C18, C19, C8, D3, D6, D8, J2, J4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

Commit message: pcb edits
Parts:
- removed C11, C12: 10u, Capacitor_SMD:C_2220_5750Metric, symbol Device:C_Small
- removed C17: 10u, Capacitor_SMD:C_0603_1608Metric_Pad1.08x0.95mm_HandSolder, symbol Device:C_Polarized
- removed C18: 22u, Capacitor_SMD:C_0603_1608Metric_Pad1.08x0.95mm_HandSolder, symbol Device:C_Polarized
- removed C37: 2.2n, Capacitor_SMD:C_0402_1005Metric, symbol Device:C_Small
- removed C40: 100n, Capacitor_SMD:C_0402_1005Metric, symbol Device:C_Small
- removed C41, C42, C43: 22u, Capacitor_SMD:C_0805_2012Metric, symbol Device:C_Small
- removed C9: 220u, Capacitor_SMD:C_1210_3225Metric, symbol Device:C_Polarized
- removed D4, D6, D7: Red LED, LED_SMD:LED_0603_1608Metric, symbol Device:LED
- removed J2: 173010542, Connector_PinHeader_2.54mm:PinHeader_1x03_P2.54mm_Vertical, symbol 173010542_5V_Buck:173010542
- removed L2: 4.7u, MainBoard:PA5432.472NLT, symbol Device:L_Small
- removed R2: 200k, Resistor_SMD:R_0402_1005Metric, symbol Device:R_Small
- removed R29: 19.6k, Resistor_SMD:R_0402_1005Metric, symbol Device:R_Small
- removed R30: 12.1k, Resistor_SMD:R_0402_1005Metric, symbol Device:R_Small
- removed R31: 1.5k, Resistor_SMD:R_0402_1005Metric, symbol Device:R_Small
- removed R4, R8: 390, Resistor_SMD:R_0402_1005Metric, symbol Device:R_Small
- removed R9: 680, Resistor_SMD:R_0402_1005Metric, symbol Device:R_Small
- removed TP2: 7.5V, TestPoint:TestPoint_Pad_D2.0mm, symbol Connector:TestPoint
- removed TP3: 5V, TestPoint:TestPoint_Pad_D2.0mm, symbol Connector:TestPoint
- removed TP4: 3.3V, TestPoint:TestPoint_Pad_D2.0mm, symbol Connector:TestPoint
- removed U4: AZ1117-3.3, Package_TO_SOT_SMD:SOT-223-3_TabPin2, symbol Regulator_Linear:AZ1117-3.3
- removed U9: AP64500Q, Package_SO:SOIC-8-1EP_3.9x4.9mm_P1.27mm_EP2.95x4.9mm_Mask2.71x3.4mm, symbol Custom:AP64500Q
- added BU33SD5WG-TR1: LM1117DT-3.3, Package_TO_SOT_SMD:SOT-23-5, symbol Regulator_Linear:MCP1802x-xx02xOT
- added C102: 1u, Capacitor_SMD:C_0603_1608Metric, symbol Device:C_Small
- added C103: 47u, Capacitor_SMD:C_0805_2012Metric, symbol Device:C_Small
- added C17, C18: 1u, Capacitor_SMD:C_0603_1608Metric_Pad1.08x0.95mm_HandSolder, symbol Device:C_Small
- added C404: 2u2, Capacitor_SMD:C_0603_1608Metric, symbol Device:C_Small
- added C9: 10u, Capacitor_SMD:C_2220_5750Metric, symbol Device:C_Small
- added R101: 1k8, Resistor_SMD:R_0402_1005Metric, symbol Device:R_Small
- added R102: 20k, Resistor_SMD:R_0402_1005Metric, symbol Device:R_Small
- added R103: 2k, Resistor_SMD:R_0402_1005Metric, symbol Device:R_Small
- added R403, R404: 0R3, Resistor_SMD:R_1210_3225Metric, symbol Device:R_Small
- added TP3V3: TestPoint_Small, TestPoint:TestPoint_Pad_D1.0mm, symbol Connector:TestPoint_Small
- added TP9V1: 3.3V, TestPoint:TestPoint_Pad_D1.0mm, symbol Connector:TestPoint
- added U101: WPME-VDLM, CustomLibrary:WPME-VDLM, symbol Custom:Buck171013801
- C10, C8: footprint Capacitor_SMD:C_1210_3225Metric -> Capacitor_SMD:C_Elec_10x10.2; MFR 885 012 209 043 -> 865060657012
- J1: footprint Connector_AMASS:AMASS_XT30PW-M_1x02_P2.50mm_Horizontal -> Connector_AMASS:AMASS_XT30UPB-F_1x02_P5.0mm_Vertical
- U1: footprint Package_SO:TSSOP-16-1EP_4.4x5mm_P0.65mm_EP3x3mm -> Package_SO:TSSOP-16_4.4x5mm_P0.65mm
Connections:
- net +7.5V is gone; now on net +9V: U1.12 (VDD)
- net +3.3V: now also BU33SD5WG-TR1.5 (VOUT), C18.1, TP3V3.1
- net ARM_B: now also R404.1; no longer U1.15 (BHS)
- net ARM_IN_A: now also R403.1; no longer U1.10 (AHS)
- net GND: now also BT1.1 (-), BU33SD5WG-TR1.2 (GND), C102.2, C103.2, C17.2, C18.2, C404.2, C9.2, R101.2, R103.2, U101.10 (AGND), U101.13 (PGND); no longer BT1.2 (-)
- net VBUS: now also C9.1, U101.4 (VIN), U101.5 (VIN)
- net at U2.1 (IP+), U2.2 (IP+): now also BT1.2 (+); no longer BT1.1 (+)
- net +5V renamed +9V
- net +9V: now also BU33SD5WG-TR1.1 (VIN), BU33SD5WG-TR1.3 (~{SHDN}), C103.1, C17.1, C404.1, R102.1, TP9V1.1, U101.6 (VOUT), U101.7 (VOUT)
- net In_A_L: no longer names the net of U1.5 (ALI)
- net In_B_L: no longer names the net of U1.4 (BLI)
- new net: R404.2, U1.15 (BHS)
- new net: R101.1, U101.1 (FSW)
- new net: R403.2, U1.10 (AHS)
- new net: U101.12 (EN), U101.9 (VIN)
- new net: R102.2, R103.1, U101.2 (FB)
- new net: C102.1, U101.3 (VCC)
- no-connect marks 9 -> 12
Other:
- sheet MCU_STM32G475 renamed MCU_STM32G474
- sheet MCU_STM32G474 ports: added IC_PWM_U_H, IC_PWM_V_H; removed IC_PWN_U_H, IC_PWN_U_L, IC_PWN_V_H, IC_PWN_V_L
- note added: "Vmax = 25.2V VBus_sense = 1.91V max"
- note added: "Wurth Capacitor : 865060657012 220uF/50V"
- note removed: "Based on Wurth 173010542 Vin : 7V-42V Vout : 5V Max : 1A"
- note removed: "Vmax = 29.6V VBus_sense = 3.3V max"
- note removed: "Wurth Capacitor : 885 012 209 043 220uF/50V"
- moved on the sheet: C19, C2, C3, C8, D1, D3, D5, D8, H109, J3, R1, R10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
