File: 2A/Hardware/Hardware_électronique/Auxiliairy_board/PCB_Moteur/Inverter_KiCAD/MCU_STM32G474.kicad_sch (KiCad schematic)
At the start: 41 parts, among them J6 Conn_ST_STDC14, J7 Conn_01x04_Pin, SW1 SW_Push, SW2 SW_Push, SW7 SW_Push, SW8 SW_Push, U6 STM32G474RETx, Y1 16M

Commit message: pcb edits
Parts:
- added TPBOOT0-1: TestPoint_Small, TestPoint:TestPoint_Pad_D1.0mm, symbol Connector:TestPoint_Small
Connections:
- net Bus_Imes: now also U6.9 (PC1); no longer U6.36 (PB14)
- net ENC_A: now also U6.12 (PA0); no longer U6.8 (PC0)
- net ENC_B: now also U6.13 (PA1); no longer U6.9 (PC1)
- net ENC_Z: now also U6.19 (PA5); no longer U6.10 (PC2)
- net ISO_PWM_Fan: now also U6.25 (PB1); no longer U6.57 (PB4)
- net PwrEn: now also U6.11 (PC3); no longer U6.2 (PC13)
- net USR_BTN_2: now also U6.57 (PB4); no longer U6.18 (PA4)
- net USR_BTN_3: now also U6.58 (PB5); no longer U6.59 (PB6)
- net U_Imes: now also U6.26 (PB2); no longer U6.13 (PA1)
- net at R15.1, U6.61 (PB8): now also TPBOOT0-1.1
- net IC_PWM_V_H: now reaches U6.21 (PA7)
- net IC_PWN_U_H: no longer names the net of U6.14 (PA2)
- net IC_PWN_U_L: no longer names the net of U6.17 (PA3)
- net IC_PWN_V_H: no longer names the net of U6.38 (PC6)
- net IC_PWN_V_L: no longer names the net of U6.39 (PC7)
- new net IC_PWM_U_H: U6.8 (PC0)
- no-connect marks 23 -> 25
