File: 2A/Hardware/Hardware_électronique/MainBoard/PCB_test/MainBoard_test1/stm32.kicad_sch (KiCad schematic)
At the start: 81 parts, among them J2 Conn_ST_STDC14, SW1 SW_Push, SW2 SW_Push, SW3 SW_Push, SW4 SW_Push, U1 STM32H735IGTx, U4 AZ1117-3.3

Commit message: Mainboard v2
Parts:
- removed C37: 10u, Capacitor_SMD:C_0805_2012Metric, symbol Device:C_Polarized
- removed C38: 22u, Capacitor_SMD:C_0402_1005Metric, symbol Device:C_Polarized
- added C10: 22u, Capacitor_SMD:C_0805_2012Metric, symbol Device:C_Small
- added C9: 10u, Capacitor_SMD:C_0805_2012Metric, symbol Device:C_Small
Connections:
- net +3.3V: now also C10.1
- net +5V: now also C9.1
- net GND: now also C10.2, C9.2
- net USB_DM: no longer names the net of U1.131 (PA12)
- net USB_DP: no longer names the net of U1.130 (PA11)
- no-connect marks 95 -> 97

Commit message: Mainboard v3
Parts:
- added C11: 220p, Capacitor_SMD:C_0402_1005Metric, symbol Device:C_Small
- added C37, C38, C48, C49: 10u, Capacitor_SMD:C_0603_1608Metric, symbol Device:C_Small
- added L2: 2u2, MainBoard:IHLL-0806AZ-1Z, symbol Device:L_Small
- C45: value 1u -> 10u; footprint Capacitor_SMD:C_0402_1005Metric -> Capacitor_SMD:C_0603_1608Metric; MFR 885 012 105 012 -> (none)
- C46: value 1u -> 4u7; MFR 885 012 105 012 -> 885 012 105 018
- C47: value 1u -> 10u; footprint Capacitor_SMD:C_0402_1005Metric -> Capacitor_SMD:C_0603_1608Metric; Fournisseur Wurth -> (none); MFR 885 012 105 012 -> (none)
Connections:
- net +3.3V: now also U1.16 (VDDSMPS), U1.17 (VFBSMPS), C37.1, C38.1, C49.1, L2.2
- net GND: now also C11.1, C37.2, C38.2, C48.2, C49.2
- net at U1.15 (VLXSMPS): now also C11.2, L2.1
- net at C42.1, U1.80 (VCAP): now also C48.1
- no-connect marks 97 -> 94
Other:
- moved on the sheet: C45

Commit message: PCB v3
Parts:
- removed C11: 220p, Capacitor_SMD:C_0402_1005Metric, symbol Device:C_Small
- removed C46: 4u7, Capacitor_SMD:C_0402_1005Metric, symbol Device:C_Small
- removed C47, C49: 10u, Capacitor_SMD:C_0603_1608Metric, symbol Device:C_Small
- removed L2: 2u2, MainBoard:IHLL-0806AZ-1Z, symbol Device:L_Small
- removed L3: 39n, Inductor_SMD:L_0603_1608Metric, symbol Device:L_Small
- added R4: 10k, Resistor_SMD:R_0402_1005Metric, symbol Device:R_Small
Connections:
- net +3.3V: now also C34.1, C35.1, U1.40 (VDDA); no longer U1.16 (VDDSMPS), U1.17 (VFBSMPS)
- net +3.3VA: no longer C34.1, C35.1, U1.40 (VDDA)
- net BOOT0: now also R4.2
- net GND: now also U1.15 (VLXSMPS), U1.16 (VDDSMPS), U1.17 (VFBSMPS), R4.1

Commit message: didn't save lol
Connections:
- net +3.3VA is gone; now on net +3.3V: C36.1, U1.39 (VREF+)

Commit message: pcb edits
Parts:
- removed C10: 22u, Capacitor_SMD:C_0805_2012Metric, symbol Device:C_Small
- removed C9: 10u, Capacitor_SMD:C_0805_2012Metric, symbol Device:C_Small
- removed TP5: TestPoint, TestPoint:TestPoint_Pad_D2.0mm, symbol Connector:TestPoint
- removed U4: AZ1117-3.3, Package_TO_SOT_SMD:SOT-223-3_TabPin2, symbol Regulator_Linear:AZ1117-3.3
Other:
- note removed: "LDO +5V-> +3.3V"
Changed lines of the file:
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@@
 (kicad_sch
-	(version 20231120)
+	(version 20250114)
 	(generator "eeschema")
-	(generator_version "8.0")
+	(generator_version "9.0")
 	(paper "A2")
