File: 2A/Hardware/Hardware_électronique/MainBoard/PCB_test/MainBoard_test1/test1.kicad_pcb (KiCad board)
At the start: 4 copper layers, 75 x 56 mm, 109 parts, among them J2 Conn_ST_STDC14, J3 Conn_02x10_Odd_Even, Q1 PMOS, SW1 SW_Push, SW2 SW_Push, SW3 SW_Push, SW4 SW_Push, U1 STM32H735IGTx, U4 AZ1117-3.3

Commit message: Mainboard v2
Parts:
- removed C37: 10u, Capacitor_SMD:C_0805_2012Metric
- removed C38: 22u, Capacitor_SMD:C_0402_1005Metric
- added C10: 22u, Capacitor_SMD:C_0805_2012Metric, B.Cu at (71.5, 65.5)
- added C9: 10u, Capacitor_SMD:C_0805_2012Metric, B.Cu at (63.5, 67.0)
- C4, C6, C8: footprint Capacitor_SMD:C_0402_1005Metric -> Capacitor_SMD:C_0805_2012Metric
- H1, H2, H3, H4: footprint MountingHole:MountingHole_2.7mm_M2.5 -> MountingHole:MountingHole_2.7mm_M2.5_DIN965_Pad
- U3: value ~ -> AP64500Q
- moved H3 48.0 mm to (110.5, 102.0)
- moved H4 48.0 mm to (110.5, 54.0)
- moved C4 3.40 mm to (59.0, 87.0)
- moved C8 2.30 mm to (62.0, 87.0)
- moved C6 0.70 mm to (65.5, 87.0)

Commit message: last minute update
Parts:
- BT1: footprint Connector_AMASS:AMASS_XT60PW-F_1x02_P7.20mm_Horizontal -> Connector_AMASS:AMASS_XT60-F_1x02_P7.20mm_Vertical; moved to F.Cu
- moved C2 1.70 mm to (57.0, 81.3)
- moved BT1 1.68 mm to (46.5, 92.7), turned to 90 degrees
- moved C7 1.63 mm to (54.8, 81.3)
- moved R1 1.36 mm to (52.6, 78.8)
- moved TP3 1.08 mm to (60.4, 65.5)
- moved D8 0.20 mm to (82.5, 62.2)
- renumbered TP5 to 3.3V
Connections:
- ARU1 pad 1: Net-(ARU1-Pad1) -> +BATT
- ARU1 pad 2: +BATT -> Net-(D10-A2)
- D10 pad 2: +BATT -> Net-(D10-A2)
- F1 pad 2: Net-(ARU1-Pad1) -> +BATT
- Q1 pad 2: +BATT -> Net-(D10-A2)
- U1 pad 130: /STM32H735/USB_DP -> unconnected-(U1-PA11-Pad130)
- U1 pad 131: /STM32H735/USB_DM -> unconnected-(U1-PA12-Pad131)
Routing:
- net Net-(D11-A): track 4.66 -> 3.20 mm
- net GND: track 49.3 -> 48.5 mm, vias 443 -> 449
- added copper zone on B.Cu, net Net-(D10-A2)
- removed copper zone on B.Cu, net Net-(ARU1-Pad1)

Commit message: Mainboard v3
Parts:
- added C11: 220p, Capacitor_SMD:C_0402_1005Metric, B.Cu at (84.0, 94.6)
- added C37: 10u, Capacitor_SMD:C_0603_1608Metric, F.Cu at (104.8, 72.8)
- added C38: 10u, Capacitor_SMD:C_0603_1608Metric, F.Cu at (73.2, 89.7)
- added C48: 10u, Capacitor_SMD:C_0603_1608Metric, B.Cu at (104.3, 75.7)
- added C49: 10u, Capacitor_SMD:C_0603_1608Metric, B.Cu at (87.8, 96.6)
- added G***1: LOGO, PCBAres:logo, B.Cu at (89.0, 79.0)
- added L2: 2u2, MainBoard:IHLL-0806AZ-1Z, B.Cu at (84.0, 96.4)
- C45: value 1u -> 10u; footprint Capacitor_SMD:C_0402_1005Metric -> Capacitor_SMD:C_0603_1608Metric
- C46: value 1u -> 4u7; moved to B.Cu
- C47: value 1u -> 10u; footprint Capacitor_SMD:C_0402_1005Metric -> Capacitor_SMD:C_0603_1608Metric; moved to B.Cu
- moved C47 27.6 mm to (87.8, 95.0)
- moved C46 14.3 mm to (85.7, 96.9), turned to -90 degrees
- moved C21 0.85 mm to (84.0, 95.4)
- moved C12 0.58 mm to (82.0, 95.4)
- moved C43 0.54 mm to (74.2, 68.9)
- moved C15 0.51 mm to (104.6, 71.5)
- moved C45 0.42 mm to (73.6, 70.4)
- moved C25 0.39 mm to (73.7, 71.7)
- moved C17 0.35 mm to (80.0, 95.4)
- moved C42 0.20 mm to (104.3, 74.2)
- renumbered 3.3V to TP3V3, TP3 to TP5V, TP1 to TPVBUS
Connections:
- U1 pad 15: unconnected-(U1-VLXSMPS-Pad15) -> Net-(U1-VLXSMPS)
- U1 pad 16: unconnected-(U1-VDDSMPS-Pad16) -> +3.3V
- U1 pad 17: unconnected-(U1-VFBSMPS-Pad17) -> +3.3V
Routing:
- net +3.3V: track 82.7 -> 99.2 mm, vias 31 -> 35
- net GND: track 48.5 -> 53.7 mm, vias 449 -> 453
- net Net-(U1-VLXSMPS): track 0.00 -> 3.65 mm, vias 0 -> 1
- net +5V: track 23.3 -> 26.5 mm
- net Net-(C42-Pad1): track 2.16 -> 4.12 mm, vias 0 -> 1
- net /STM32H735/USR_LED_3: track 44.9 -> 45.7 mm
- net /STM32H735/USR_LED_4: track 42.6 -> 43.4 mm
- net /STM32H735/USR_LED_1: track 47.1 -> 47.9 mm
- net /STM32H735/USR_LED_2: track 45.6 -> 46.3 mm
Other:
- board text added: "PCB_MainBoard_v3 By Kenny Saint Fleur"

Commit message: PCB v3
Parts:
- removed C11: 220p, Capacitor_SMD:C_0402_1005Metric
- removed C46: 4u7, Capacitor_SMD:C_0402_1005Metric
- removed C47, C49: 10u, Capacitor_SMD:C_0603_1608Metric
- removed L2: 2u2, MainBoard:IHLL-0806AZ-1Z
- removed L3: 39n, Inductor_SMD:L_0603_1608Metric
- added R4: 10k, Resistor_SMD:R_0402_1005Metric, B.Cu at (73.4, 87.7)
- C34, C35, C36: moved to F.Cu
- moved C35 0.95 mm to (95.6, 96.4), turned to -90 degrees
- moved C34 0.85 mm to (94.5, 96.4), turned to -90 degrees
- moved C36 0.60 mm to (96.7, 96.4), turned to -90 degrees
- moved C39 0.55 mm to (93.3, 96.5)
- renumbered TPVBUS to TP1, TP5V to TP3, TP3V3 to TP5
Connections:
- C34 pad 1: +3.3VA -> +3.3V
- C35 pad 1: +3.3VA -> +3.3V
- C36 pad 1: +3.3VA -> +3.3V
- U1 pad 15: Net-(U1-VLXSMPS) -> GND
- U1 pad 16: +3.3V -> GND
- U1 pad 17: +3.3V -> GND
- U1 pad 39: +3.3VA -> +3.3V
- U1 pad 40: +3.3VA -> +3.3V
Routing:
- net +3.3V: track 99.2 -> 94.8 mm
- net Net-(U1-VLXSMPS): track 3.65 -> 0.00 mm, vias 1 -> 0
- net +3.3VA: track 3.62 -> 0.00 mm, vias 1 -> 0
- net /STM32H735/TX4: track 24.6 -> 26.4 mm
- net GND: track 53.7 -> 55.4 mm, vias 453 -> 455
- net /STM32H735/RX4: track 22.7 -> 24.3 mm
- net /GPIO14_TXD: track 22.2 -> 21.5 mm
- net /STM32H735/NRST: track 51.3 -> 51.8 mm
- net /STM32H735/BOOT0: track 5.78 -> 6.22 mm, vias 0 -> 1
- removed copper zone on B.Cu, net +3.3VA

Commit message: last details
Routing:
- net GND: track 55.4 -> 76.1 mm, vias 455 -> 470

Commit message: pcb edits
Parts:
- removed C10, C4, C6, C8: 22u, Capacitor_SMD:C_0805_2012Metric
- removed C2, C7, C9: 10u, Capacitor_SMD:C_0805_2012Metric
- removed C3: 2.2n, Capacitor_SMD:C_0402_1005Metric
- removed C5: 100n, Capacitor_SMD:C_0402_1005Metric
- removed L1: 4.7u, MainBoard:PA5432.472NLT
- removed R2: 200k, Resistor_SMD:R_0402_1005Metric
- removed R3: 19.6k, Resistor_SMD:R_0402_1005Metric
- removed R5: 36k, Resistor_SMD:R_0402_1005Metric
- removed R6: 6.8k, Resistor_SMD:R_0402_1005Metric
- removed TP1, TP3: TestPoint, TestPoint:TestPoint_Pad_D2.0mm
- removed U3: AP64500Q, Package_SO:SOIC-8-1EP_3.9x4.9mm_P1.27mm_EP2.95x4.9mm_Mask2.71x3.4mm
- removed U4: AZ1117-3.3, Package_TO_SOT_SMD:SOT-223-3_TabPin2
- added C11: 10u, Capacitor_SMD:C_0805_2012Metric, B.Cu at (56.8, 79.8)
- added C46: 1u, Capacitor_SMD:C_0603_1608Metric, B.Cu at (64.0, 76.5)
- added C47: 47u, Capacitor_SMD:C_0805_2012Metric, B.Cu at (69.3, 76.2)
- added J1: 173010542, Connector_PinHeader_2.54mm:PinHeader_1x03_P2.54mm_Vertical, F.Cu at (93.4, 52.9)
- added R7: 1k8, Resistor_SMD:R_0402_1005Metric, B.Cu at (59.1, 76.5)
- added R8: 7k5, Resistor_SMD:R_0402_1005Metric, B.Cu at (60.3, 76.5)
- added R9: 2k7, Resistor_SMD:R_0402_1005Metric, B.Cu at (61.4, 76.5)
- added TP3V3: 3.3V, TestPoint:TestPoint_Pad_D1.0mm, B.Cu at (68.4, 85.0)
- added TP5V1: 3.3V, TestPoint:TestPoint_Pad_D1.0mm, B.Cu at (88.3, 56.8)
- added TPVBUS1: 3.3V, TestPoint:TestPoint_Pad_D1.0mm, F.Cu at (56.3, 74.0)
- added U2: WPME-VDLM, CustomLibrary:WPME-VDLM, B.Cu at (64.3, 80.7)
- moved D10 2.33 mm to (59.8, 70.3), turned to -90 degrees
- moved R4 1.65 mm to (75.0, 88.1)
- moved TP5 0.70 mm to (70.2, 93.0)
Connections:
- J3 pad 2: +5V -> unconnected-(J3-Pin_2-Pad2)
- J3 pad 4: +5V -> unconnected-(J3-Pin_4-Pad4)
Routing:
- net Net-(U3-SW): track 16.1 -> 0.00 mm
- net GND: track 76.1 -> 88.7 mm, vias 470 -> 461
- net +3.3V: track 94.8 -> 100.9 mm, vias 35 -> 40
- net +5V: track 26.5 -> 22.2 mm, vias 16 -> 1
- net Net-(U2-EN): track 0.00 -> 3.46 mm
- net /STM32H735/RX8: track 16.0 -> 19.1 mm
- net Net-(U3-FB): track 2.84 -> 0.00 mm
- net Net-(U2-VCC): track 0.00 -> 2.36 mm
- net Net-(C3-Pad1): track 1.87 -> 0.00 mm
- net Net-(U3-BST): track 1.74 -> 0.00 mm
- net Net-(U3-COMP): track 1.70 -> 0.00 mm
- net Net-(U2-FSW): track 0.00 -> 1.50 mm
- net Net-(U3-RT/CLK): track 1.46 -> 0.00 mm
- net /STM32H735/RX10: track 19.0 -> 17.7 mm
- net /STM32H735/BOOT0: track 6.22 -> 7.13 mm
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- added copper zone on B.Cu, net Net-(U2-FB)
- removed copper zone on B.Cu, net +5V
- removed copper zone on In2.Cu, net +5V
- removed copper zone on B.Cu, net Net-(U3-FB)
- removed copper zone on B.Cu, net Net-(U3-SW)
Other:
- board text added: "PCB_MainBoard_v4 By Kenny Saint Fleur"
- board text removed: "PCB_MainBoard_v3 By Kenny Saint Fleur"
